File: actidamp-mk4-smd.sch (KiCad schematic (older format))
At the start: 22 parts

Commit message: Move stuff to hierarchy
Parts:
- removed C? (x8): C, symbol Device:C
- removed L?: L, symbol Device:L
- removed Q? (x2): Q_NJFET_DGS, symbol Device:Q_NJFET_DGS
- removed R? (x8): R, symbol Device:R
- removed SW?: SW_DIP_x04, symbol Switch:SW_DIP_x04
- removed U? (x2): NE5534, symbol Amplifier_Operational:NE5534
Connections:
- net labels removed: GND
- wire segments 58 -> 0

Commit message: Capture of original actidamp iv
Parts:
- added J? (x4): Screw_Terminal_01x02, symbol Connector:Screw_Terminal_01x02
Connections:
- net labels added: GND
- wire segments 0 -> 12
Changed lines of the file:
@@
 $Descr A4 11693 8268
 encoding utf-8
-Sheet 1 2
+Sheet 1 3
 Title ""
 Date ""
@@
 $EndDescr
 $Sheet
-S 8950 5000 1050 800
+S 4750 2550 1050 400
 U 5C72F90C
-F0 "channel" 50
+F0 "left_channel" 50
 F1 "channel.sch" 50
+F2 "IN" I L 4750 2750 50
+F3 "OUT" O R 5800 2750 50
 $EndSheet
+$Comp
+L Connector:Screw_Terminal_01x02 J?
+U 1 1 5C7377B7
+P 3850 2850
+F 0 "J?" H 3770 2525 50  0000 C CNN
+F 1 "Screw_Terminal_01x02" H 3770 2616 50  0000 C CNN
+F 2 "" H 3850 2850 50  0001 C CNN
+F 3 "~" H 3850 2850 50  0001 C CNN
+	1    3850 2850
+	-1   0    0    1
+$EndComp
+Wire Wire Line
+	4050 2750 4750 2750
+$Comp
+L power:GND #PWR?
+U 1 1 5C737820
+P 4550 2950
+F 0 "#PWR?" H 4550 2700 50  0001 C CNN
+F 1 "GND" H 4555 2777 50  0000 C CNN
+F 2 "" H 4550 2950 50  0001 C CNN
+F 3 "" H 4550 2950 50  0001 C CNN
+	1    4550 2950
+	1    0    0    -1
+$EndComp
+Wire Wire Line
+	4050 2850 4550 2850
+Wire Wire Line
+	4550 2850 4550 2950
+$Comp
+L power:GND #PWR?
+U 1 1 5C73784D
+P 6050 2950
+F 0 "#PWR?" H 6050 2700 50  0001 C CNN
+F 1 "GND" H 6055 2777 50  0000 C CNN
+F 2 "" H 6050 2950 50  0001 C CNN
+F 3 "" H 6050 2950 50  0001 C CNN
+	1    6050 2950
+	1    0    0    -1
+$EndComp
+$Comp
+L Connector:Screw_Terminal_01x02 J?
+U 1 1 5C73787D
+P 6750 2750
+F 0 "J?" H 6830 2742 50  0000 L CNN
+F 1 "Screw_Terminal_01x02" H 6830 2651 50  0000 L CNN
+F 2 "" H 6750 2750 50  0001 C CNN
+F 3 "~" H 6750 2750 50  0001 C CNN
+	1    6750 2750
+	1    0    0    -1
+$EndComp
+Wire Wire Line
+	5800 2750 6550 2750
+Wire Wire Line
+	6050 2950 6050 2850
+Wire Wire Line
+	6050 2850 6550 2850
+$Sheet
+S 4750 3500 1050 400
+U 5C7379E1
+F0 "right_channel" 50
+F1 "channel.sch" 50
+F2 "IN" I L 4750 3700 50
+F3 "OUT" O R 5800 3700 50
+$EndSheet
+$Comp
+L Connector:Screw_Terminal_01x02 J?
+U 1 1 5C7379E7
+P 3850 3800
+F 0 "J?" H 3770 3475 50  0000 C CNN
+F 1 "Screw_Terminal_01x02" H 3770 3566 50  0000 C CNN
+F 2 "" H 3850 3800 50  0001 C CNN
+F 3 "~" H 3850 3800 50  0001 C CNN
+	1    3850 3800
+	-1   0    0    1
+$EndComp
+Wire Wire Line
+	4050 3700 4750 3700
+$Comp
+L power:GND #PWR?
+U 1 1 5C7379EF
+P 4550 3900
+F 0 "#PWR?" H 4550 3650 50  0001 C CNN
+F 1 "GND" H 4555 3727 50  0000 C CNN
+F 2 "" H 4550 3900 50  0001 C CNN
+F 3 "" H 4550 3900 50  0001 C CNN
+	1    4550 3900
+	1    0    0    -1
+$EndComp
+Wire Wire Line
+	4050 3800 4550 3800
+Wire Wire Line
+	4550 3800 4550 3900
+$Comp
+L power:GND #PWR?
+U 1 1 5C7379F7
+P 6050 3900
+F 0 "#PWR?" H 6050 3650 50  0001 C CNN
+F 1 "GND" H 6055 3727 50  0000 C CNN
+F 2 "" H 6050 3900 50  0001 C CNN
+F 3 "" H 6050 3900 50  0001 C CNN
+	1    6050 3900
+	1    0    0    -1
+$EndComp
+$Comp
+L Connector:Screw_Terminal_01x02 J?
+U 1 1 5C7379FD
+P 6750 3700
+F 0 "J?" H 6830 3692 50  0000 L CNN
+F 1 "Screw_Terminal_01x02" H 6830 3601 50  0000 L CNN
+F 2 "" H 6750 3700 50  0001 C CNN
+F 3 "~" H 6750 3700 50  0001 C CNN
+	1    6750 3700
+	1    0    0    -1
+$EndComp
+Wire Wire Line
+	5800 3700 6550 3700
+Wire Wire Line
+	6050 3900 6050 3800
+Wire Wire Line
+	6050 3800 6550 3800
 $EndSCHEMATC

Commit message: Assign capacitors, redo hierarchy
Parts:
- removed J? (x4): Screw_Terminal_01x02, symbol Connector:Screw_Terminal_01x02
- added J? (x2): Screw_Terminal_01x03, symbol Connector:Screw_Terminal_01x03
Connections:
- wire segments 12 -> 14
Changed lines of the file:
@@
 F0 "left_channel" 50
 F1 "channel.sch" 50
-F2 "IN" I L 4750 2750 50
+F2 "IN" I L 4750 2850 50
 F3 "OUT" O R 5800 2750 50
+F4 "V+" I L 4750 2600 50
+F5 "V-" I L 4750 2700 50
+$EndSheet
+$Sheet
+S 4750 3150 1050 400
+U 5C7379E1
+F0 "right_channel" 50
+F1 "channel.sch" 50
+F2 "IN" I L 4750 3250 50
+F3 "OUT" O R 5800 3350 50
+F4 "V+" I L 4750 3400 50
+F5 "V-" I L 4750 3500 50
 $EndSheet
 $Comp
-L Connector:Screw_Terminal_01x02 J?
-U 1 1 5C7377B7
-P 3850 2850
-F 0 "J?" H 3770 2525 50  0000 C CNN
-F 1 "Screw_Terminal_01x02" H 3770 2616 50  0000 C CNN
-F 2 "" H 3850 2850 50  0001 C CNN
-F 3 "~" H 3850 2850 50  0001 C CNN
-	1    3850 2850
-	-1   0    0    1
-$EndComp
-Wire Wire Line
-	4050 2750 4750 2750
-$Comp
-L power:GND #PWR?
-U 1 1 5C737820
-P 4550 2950
-F 0 "#PWR?" H 4550 2700 50  0001 C CNN
-F 1 "GND" H 4555 2777 50  0000 C CNN
-F 2 "" H 4550 2950 50  0001 C CNN
-F 3 "" H 4550 2950 50  0001 C CNN
-	1    4550 2950
-	1    0    0    -1
-$EndComp
-Wire Wire Line
-	4050 2850 4550 2850
-Wire Wire Line
-	4550 2850 4550 2950
-$Comp
-L power:GND #PWR?
-U 1 1 5C73784D
-P 6050 2950
-F 0 "#PWR?" H 6050 2700 50  0001 C CNN
-F 1 "GND" H 6055 2777 50  0000 C CNN
-F 2 "" H 6050 2950 50  0001 C CNN
-F 3 "" H 6050 2950 50  0001 C CNN
-	1    6050 2950
+L Connector:Screw_Terminal_01x03 J?
+U 1 1 5D89132C
+P 6350 3050
+F 0 "J?" H 6430 3092 50  0000 L CNN
+F 1 "Screw_Terminal_01x03" H 6430 3001 50  0000 L CNN
+F 2 "" H 6350 3050 50  0001 C CNN
+F 3 "~" H 6350 3050 50  0001 C CNN
+	1    6350 3050
 	1    0    0    -1
 $EndComp
 $Comp
-L Connector:Screw_Terminal_01x02 J?
-U 1 1 5C73787D
-P 6750 2750
-F 0 "J?" H 6830 2742 50  0000 L CNN
-F 1 "Screw_Terminal_01x02" H 6830 2651 50  0000 L CNN
-F 2 "" H 6750 2750 50  0001 C CNN
-F 3 "~" H 6750 2750 50  0001 C CNN
-	1    6750 2750
-	1    0    0    -1
+L Connector:Screw_Terminal_01x03 J?
+U 1 1 5D89140D
+P 4150 3050
+F 0 "J?" H 4700 3100 50  0000 C CNN
+F 1 "Screw_Terminal_01x03" H 4700 3000 50  0000 C CNN
+F 2 "" H 4150 3050 50  0001 C CNN
+F 3 "~" H 4150 3050 50  0001 C CNN
+	1    4150 3050
+	-1   0    0    -1
 $EndComp
 Wire Wire Line
-	5800 2750 6550 2750
+	5800 2750 6000 2750
 Wire Wire Line
-	6050 2950 6050 2850
+	6000 2750 6000 2950
 Wire Wire Line
-	6050 2850 6550 2850
-$Sheet
-S 4750 3500 1050 400
-U 5C7379E1
-F0 "right_channel" 50
-F1 "channel.sch" 50
-F2 "IN" I L 4750 3700 50
-F3 "OUT" O R 5800 3700 50
-$EndSheet
+	6000 2950 6150 2950
+Wire Wire Line
+	4350 2950 4550 2950
+Wire Wire Line
+	4350 3150 4550 3150
+Wire Wire Line
+	6150 3150 6000 3150
+Wire Wire Line
+	6000 3150 6000 3350
+Wire Wire Line
+	6000 3350 5800 3350
 $Comp
-L Connector:Screw_Terminal_01x02 J?
-U 1 1 5C7379E7
-P 3850 3800
-F 0 "J?" H 3770 3475 50  0000 C CNN
-F 1 "Screw_Terminal_01x02" H 3770 3566 50  0000 C CNN
-F 2 "" H 3850 3800 50  0001 C CNN
-F 3 "~" H 3850 3800 50  0001 C CNN
-	1    3850 3800
-	-1   0    0    1
+L power:GND #PWR?
+U 1 1 5D89189D
+P 6100 3050
+F 0 "#PWR?" H 6100 2800 50  0001 C CNN
+F 1 "GND" V 6105 2922 50  0000 R CNN
+F 2 "" H 6100 3050 50  0001 C CNN
+F 3 "" H 6100 3050 50  0001 C CNN
+	1    6100 3050
+	0    1    1    0
+$EndComp
+$Comp
+L power:GND #PWR?
+U 1 1 5D8919EB
+P 4400 3050
+F 0 "#PWR?" H 4400 2800 50  0001 C CNN
+F 1 "GND" V 4405 2922 50  0000 R CNN
+F 2 "" H 4400 3050 50  0001 C CNN
+F 3 "" H 4400 3050 50  0001 C CNN
+	1    4400 3050
+	0    -1   -1   0
 $EndComp
 Wire Wire Line
-	4050 3700 4750 3700
-$Comp
-L power:GND #PWR?
-U 1 1 5C7379EF
-P 4550 3900
-F 0 "#PWR?" H 4550 3650 50  0001 C CNN
-F 1 "GND" H 4555 3727 50  0000 C CNN
-F 2 "" H 4550 3900 50  0001 C CNN
-F 3 "" H 4550 3900 50  0001 C CNN
-	1    4550 3900
-	1    0    0    -1
-$EndComp
+	4350 3050 4400 3050
 Wire Wire Line
-	4050 3800 4550 3800
+	6100 3050 6150 3050
 Wire Wire Line
-	4550 3800 4550 3900
-$Comp
-L power:GND #PWR?
-U 1 1 5C7379F7
-P 6050 3900
-F 0 "#PWR?" H 6050 3650 50  0001 C CNN
-F 1 "GND" H 6055 3727 50  0000 C CNN
-F 2 "" H 6050 3900 50  0001 C CNN
-F 3 "" H 6050 3900 50  0001 C CNN
-	1    6050 3900
-	1    0    0    -1
-$EndComp
-$Comp
-L Connector:Screw_Terminal_01x02 J?
-U 1 1 5C7379FD
-P 6750 3700
-F 0 "J?" H 6830 3692 50  0000 L CNN
-F 1 "Screw_Terminal_01x02" H 6830 3601 50  0000 L CNN
-F 2 "" H 6750 3700 50  0001 C CNN
-F 3 "~" H 6750 3700 50  0001 C CNN
-	1    6750 3700
-	1    0    0    -1
-$EndComp
+	4550 2950 4550 2850
 Wire Wire Line
-	5800 3700 6550 3700
+	4550 2850 4750 2850
 Wire Wire Line
-	6050 3900 6050 3800
+	4550 3150 4550 3250
 Wire Wire Line
-	6050 3800 6550 3800
+	4550 3250 4750 3250
 $EndSCHEMATC

Commit message: All schematics drafted
Parts:
- removed J? (x2): Screw_Terminal_01x03, symbol Connector:Screw_Terminal_01x03
- added C? (x4): 10u, symbol Device:CP
- added C? (x2): 220u, symbol Device:CP
- added D? (x4): D, symbol Device:D
- added J1: PHONO_IN_L, symbol Connector:Barrel_Jack_Switch
- added J2: PHONO_IN_R, symbol Connector:Barrel_Jack_Switch
- added J3: LINE_OUT_L, symbol Connector:Barrel_Jack_Switch
- added J4: LINE_OUT_R, symbol Connector:Barrel_Jack_Switch
- added J?: Phono_Ground, symbol Connector:Screw_Terminal_01x01
- added J?: Screw_Terminal_01x03, symbol Connector:Screw_Terminal_01x03
- added R? (x4): R, symbol Device:R
- added U?: LM317_3PinPackage, symbol Regulator_Linear:LM317_3PinPackage
- added U?: LM337_TO252, Package_TO_SOT_SMD:TO-252-2, symbol Regulator_Linear:LM337_TO252
Connections:
- wire segments 14 -> 85

Commit message: Finalise schematics with power supplies and successful ERC
Parts:
- removed J?: Screw_Terminal_01x03, symbol Connector:Screw_Terminal_01x03
- added H101, H102, H103, H104: MountingHole, symbol Mechanical:MountingHole
- added HS101, HS102: Heatsink_Pad, symbol Mechanical:Heatsink_Pad
- added J101: XLR3, symbol Connector:XLR3
- D101, D102: renamed from D?; Part number (none) -> MRA4003T3G
- U101: renamed from U?; Additional (none) -> FK 244 13 D PAK; Part number (none) -> LM317MDTX
- U102: renamed from U?; Part number (none) -> LM337KVURG3
- gave numbers to parts that had none: 13
- renumbered J1 to J103, J2 to J104, J3 to J105, J4 to J106
Connections:
- wire segments 85 -> 92

Commit message: Finalise BOM
Parts:
- C101, C102: Parameters (none) -> SMT Electrolytic 25V; Part number (none) -> EEE1HA221UAP
- C103, C104, C105, C106: symbol Device:CP -> Device:C; Parameters (none) -> X7R/X5R 25V 1206; Part number (none) -> C1206C106K3PACTU
- D101, D102: Parameters (none) -> 1A general purpose
- D103, D104: Parameters (none) -> 100mA general purpose; Part number (none) -> BAS20
- HS101, HS102: Parameters (none) -> SMT for TO-252
- R101, R102: value R -> 3400 1%; Parameters (none) -> Thin Film 0603; Part number (none) -> MCWF06R3401BTL
- R103, R104: value R -> 240 1%; Parameters (none) -> Thin Film 0603; Part number (none) -> ERA3AEB241V
- U101: Additional FK 244 13 D PAK -> (none); Parameters (none) -> TO-252
- U102: Parameters (none) -> TO-252
Other:
- note added: "Input in range of +-25 up to +-35V"
- note added: "The output of regulators should be +- approx. 18.5\nThat makes +- approx. 17.5 after psu_rails capacitor multiplier"
Changed lines of the file:
@@
 	5300 3350 5500 3350
 $Comp
-L Device:CP C105
+L Device:C C105
 U 1 1 5D8EA5F7
 P 4850 2700
@@
 F 2 "" H 4888 2550 50  0001 C CNN
 F 3 "~" H 4850 2700 50  0001 C CNN
+F 4 "X7R/X5R 25V 1206" H 0   0   50  0001 C CNN "Parameters"
+F 5 "C1206C106K3PACTU" H 0   0   50  0001 C CNN "Part number"
 	1    4850 2700
 	1    0    0    -1
 $EndComp
 $Comp
-L Device:CP C103
+L Device:C C103
 U 1 1 5D8EA64D
 P 4450 2700
@@
 F 2 "" H 4488 2550 50  0001 C CNN
 F 3 "~" H 4450 2700 50  0001 C CNN
+F 4 "X7R/X5R 25V 1206" H 4450 2700 50  0001 C CNN "Parameters"
+F 5 "C1206C106K3PACTU" H 0   0   50  0001 C CNN "Part number"
 	1    4450 2700
 	1    0    0    -1
@@
 F 2 "" H 3350 2750 50  0001 C CIN
 F 3 "http://www.ti.com/lit/ds/symlink/lm317.pdf" H 3350 2500 50  0001 C CNN
-F 4 "	FK 244 13 D PAK" H 0   0   50  0001 C CNN "Additional"
+F 4 "" H 0   0   50  0001 C CNN "Additional"
 F 5 "LM317MDTX" H 3350 2500 50  0001 C CNN "Part number"
+F 6 "TO-252" H 0   0   50  0001 C CNN "Parameters"
 	1    3350 2500
 	1    0    0    -1
@@
 F 3 "http://www.farnell.com/datasheets/1636957.pdf" H 3350 3950 50  0001 C CNN
 F 4 "LM337KVURG3" H 0   0   50  0001 C CNN "Part number"
+F 5 "TO-252" H 0   0   50  0001 C CNN "Parameters"
 	1    3350 3950
 	1    0    0    1
@@
 F 2 "" H 2638 2550 50  0001 C CNN
 F 3 "~" H 2600 2700 50  0001 C CNN
+F 4 "EEE1HA221UAP" H 0   0   50  0001 C CNN "Part number"
+F 5 "SMT Electrolytic 25V" H 0   0   50  0001 C CNN "Parameters"
 	1    2600 2700
 	1    0    0    -1
@@
 U 1 1 5D8F0F6F
 P 4050 2700
-F 0 "D103" V 4004 2779 50  0000 L CNN
-F 1 "D" V 4095 2779 50  0000 L CNN
+F 0 "D103" V 4350 2650 50  0000 L CNN
+F 1 "D" V 4450 2650 50  0000 L CNN
 F 2 "" H 4050 2700 50  0001 C CNN
 F 3 "~" H 4050 2700 50  0001 C CNN
+F 4 "BAS20" H 0   0   50  0001 C CNN "Part number"
+F 5 "100mA general purpose" H 0   0   50  0001 C CNN "Parameters"
 	1    4050 2700
 	0    1    1    0
@@
 U 1 1 5D8F102E
 P 3800 2700
-F 0 "R103" H 3870 2746 50  0000 L CNN
-F 1 "R" H 3870 2655 50  0000 L CNN
+F 0 "R103" H 3700 2400 50  0000 L CNN
+F 1 "240 1%" H 3700 2300 50  0000 L CNN
 F 2 "" V 3730 2700 50  0001 C CNN
 F 3 "~" H 3800 2700 50  0001 C CNN
+F 4 "ERA3AEB241V" H 0   0   50  0001 C CNN "Part number"
+F 5 "Thin Film 0603" H 0   0   50  0001 C CNN "Parameters"
 	1    3800 2700
 	1    0    0    -1
@@
 U 1 1 5D8F4A8C
 P 3350 3100
-F 0 "R101" H 3420 3146 50  0000 L CNN
-F 1 "R" H 3420 3055 50  0000 L CNN
+F 0 "R101" H 3400 3100 50  0000 L CNN
+F 1 "3400 1%" H 3400 3000 50  0000 L CNN
 F 2 "" V 3280 3100 50  0001 C CNN
 F 3 "~" H 3350 3100 50  0001 C CNN
+F 4 "MCWF06R3401BTL" H 0   0   50  0001 C CNN "Part number"
+F 5 "Thin Film 0603" H 0   0   50  0001 C CNN "Parameters"
 	1    3350 3100
 	1    0    0    -1
@@
 Wire Wire Line
 	3800 2850 3800 2900
-Connection ~ 3800 2900
 Wire Wire Line
 	3800 2900 4050 2900
@@
 F 3 "~" H 2250 2500 50  0001 C CNN
 F 4 "MRA4003T3G" H 0   0   50  0001 C CNN "Part number"
+F 5 "1A general purpose" H 0   0   50  0001 C CNN "Parameters"
 	1    2250 2500
 	-1   0    0    1
@@
 	2400 2500 2600 2500
 $Comp
-L Device:CP C106
+L Device:C C106
 U 1 1 5D8FE2B6
 P 4850 4150
@@
 F 2 "" H 4888 4000 50  0001 C CNN
 F 3 "~" H 4850 4150 50  0001 C CNN
+F 4 "X7R/X5R 25V 1206" H 0   0   50  0001 C CNN "Parameters"
+F 5 "C1206C106K3PACTU" H 0   0   50  0001 C CNN "Part number"
 	1    4850 4150
 	-1   0    0    1
 $EndComp
 $Comp
-L Device:CP C104
+L Device:C C104
 U 1 1 5D8FE2BC
 P 4450 4150
@@
 F 2 "" H 4488 4000 50  0001 C CNN
 F 3 "~" H 4450 4150 50  0001 C CNN
+F 4 "X7R/X5R 25V 1206" H 0   0   50  0001 C CNN "Parameters"
+F 5 "C1206C106K3PACTU" H 0   0   50  0001 C CNN "Part number"
 	1    4450 4150
 	-1   0    0    1
@@
 F 2 "" H 2638 4000 50  0001 C CNN
 F 3 "~" H 2600 4150 50  0001 C CNN
+F 4 "EEE1HA221UAP" H 0   0   50  0001 C CNN "Part number"
+F 5 "SMT Electrolytic 25V" H 0   0   50  0001 C CNN "Parameters"
 	1    2600 4150
 	-1   0    0    1
@@
 U 1 1 5D8FE2EB
 P 4050 4150
-F 0 "D104" V 4096 4229 50  0000 L CNN
-F 1 "D" V 4005 4229 50  0000 L CNN
+F 0 "D104" V 3750 4100 50  0000 L CNN
+F 1 "D" V 3650 4100 50  0000 L CNN
 F 2 "" H 4050 4150 50  0001 C CNN
 F 3 "~" H 4050 4150 50  0001 C CNN
+F 4 "BAS20" H 0   0   50  0001 C CNN "Part number"
+F 5 "100mA general purpose" H 0   0   50  0001 C CNN "Parameters"
 	1    4050 4150
 	0    1    -1   0
@@
 U 1 1 5D8FE2F1
 P 3800 4150
-F 0 "R104" H 3870 4196 50  0000 L CNN
-F 1 "R" H 3870 4105 50  0000 L CNN
+F 0 "R104" H 3700 3850 50  0000 L CNN
+F 1 "240 1%" H 3700 3750 50  0000 L CNN
 F 2 "" V 3730 4150 50  0001 C CNN
 F 3 "~" H 3800 4150 50  0001 C CNN
+F 4 "ERA3AEB241V" H 0   0   50  0001 C CNN "Part number"
+F 5 "Thin Film 0603" H 0   0   50  0001 C CNN "Parameters"
 	1    3800 4150
 	1    0    0    -1
@@
 U 1 1 5D8FE2FF
 P 3350 4550
-F 0 "R102" H 3420 4596 50  0000 L CNN
-F 1 "R" H 3420 4505 50  0000 L CNN
+F 0 "R102" H 3400 4550 50  0000 L CNN
+F 1 "3400 1%" H 3400 4450 50  0000 L CNN
 F 2 "" V 3280 4550 50  0001 C CNN
 F 3 "~" H 3350 4550 50  0001 C CNN
+F 4 "MCWF06R3401BTL" H 0   0   50  0001 C CNN "Part number"
+F 5 "Thin Film 0603" H 0   0   50  0001 C CNN "Parameters"
 	1    3350 4550
 	1    0    0    -1
@@
 F 3 "~" H 2250 3950 50  0001 C CNN
 F 4 "MRA4003T3G" H 0   0   50  0001 C CNN "Part number"
+F 5 "1A general purpose" H 0   0   50  0001 C CNN "Parameters"
 	1    2250 3950
 	1    0    0    1
@@
 F 3 "~" H 3812 2200 50  0001 C CNN
 F 4 "FK 244 13 D PAK" H 3800 2250 50  0001 C CNN "Part number"
+F 5 "SMT for TO-252" H 0   0   50  0001 C CNN "Parameters"
 	1    3800 2250
 	1    0    0    -1
@@
 F 3 "~" H 2612 3600 50  0001 C CNN
 F 4 "FK 244 13 D PAK" H 2600 3650 50  0001 C CNN "Part number"
+F 5 "SMT for TO-252" H 0   0   50  0001 C CNN "Parameters"
 	1    2600 3650
 	1    0    0    -1
@@
 	2100 3100 2100 3250
 Connection ~ 2100 3250
+Connection ~ 3800 2900
+Text Notes 2800 2050 0    50   ~ 0
+The output of regulators should be +- approx. 18.5\nThat makes +- approx. 17.5 after psu_rails capacitor multiplier
+Text Notes 1300 4000 1    50   ~ 0
+Input in range of +-25 up to +-35V
 $EndSCHEMATC

Commit message: WIP: Assign footprints
Parts:
- C101, C102: footprint (none) -> Capacitor_SMD:CP_Elec_8x10.5; Part number EEE1HA221UAP -> EEE1EA221UP
- C103, C104, C105, C106: footprint (none) -> Capacitor_SMD:C_1206_3216Metric_Pad1.42x1.75mm_HandSolder
- D101, D102: footprint (none) -> Diode_SMD:D_SMA
- D103, D104: footprint (none) -> Diode_SMD:D_SOT-23_ANK
- H101, H102, H103, H104: footprint (none) -> MountingHole:MountingHole_2.7mm_M2.5
- U101: footprint (none) -> Package_TO_SOT_SMD:TO-252-2
Changed lines of the file:
@@
 F 0 "C105" H 4968 2746 50  0000 L CNN
 F 1 "10u" H 4968 2655 50  0000 L CNN
-F 2 "" H 4888 2550 50  0001 C CNN
+F 2 "Capacitor_SMD:C_1206_3216Metric_Pad1.42x1.75mm_HandSolder" H 4888 2550 50  0001 C CNN
 F 3 "~" H 4850 2700 50  0001 C CNN
 F 4 "X7R/X5R 25V 1206" H 0   0   50  0001 C CNN "Parameters"
@@
 F 0 "C103" H 4568 2746 50  0000 L CNN
 F 1 "10u" H 4568 2655 50  0000 L CNN
-F 2 "" H 4488 2550 50  0001 C CNN
+F 2 "Capacitor_SMD:C_1206_3216Metric_Pad1.42x1.75mm_HandSolder" H 4488 2550 50  0001 C CNN
 F 3 "~" H 4450 2700 50  0001 C CNN
 F 4 "X7R/X5R 25V 1206" H 4450 2700 50  0001 C CNN "Parameters"
@@
 F 0 "U101" H 3350 2742 50  0000 C CNN
 F 1 "LM317_3PinPackage" H 3350 2651 50  0000 C CNN
-F 2 "" H 3350 2750 50  0001 C CIN
+F 2 "Package_TO_SOT_SMD:TO-252-2" H 3350 2750 50  0001 C CIN
 F 3 "http://www.ti.com/lit/ds/symlink/lm317.pdf" H 3350 2500 50  0001 C CNN
 F 4 "" H 0   0   50  0001 C CNN "Additional"
@@
 F 0 "C101" H 2718 2746 50  0000 L CNN
 F 1 "220u" H 2718 2655 50  0000 L CNN
-F 2 "" H 2638 2550 50  0001 C CNN
+F 2 "Capacitor_SMD:CP_Elec_8x10.5" H 2638 2550 50  0001 C CNN
 F 3 "~" H 2600 2700 50  0001 C CNN
-F 4 "EEE1HA221UAP" H 0   0   50  0001 C CNN "Part number"
+F 4 "EEE1EA221UP" H 0   0   50  0001 C CNN "Part number"
 F 5 "SMT Electrolytic 25V" H 0   0   50  0001 C CNN "Parameters"
 	1    2600 2700
@@
 F 0 "D103" V 4350 2650 50  0000 L CNN
 F 1 "D" V 4450 2650 50  0000 L CNN
-F 2 "" H 4050 2700 50  0001 C CNN
+F 2 "Diode_SMD:D_SOT-23_ANK" H 4050 2700 50  0001 C CNN
 F 3 "~" H 4050 2700 50  0001 C CNN
 F 4 "BAS20" H 0   0   50  0001 C CNN "Part number"
@@
 F 0 "D101" H 2250 2284 50  0000 C CNN
 F 1 "D" H 2250 2375 50  0000 C CNN
-F 2 "" H 2250 2500 50  0001 C CNN
+F 2 "Diode_SMD:D_SMA" H 2250 2500 50  0001 C CNN
 F 3 "~" H 2250 2500 50  0001 C CNN
 F 4 "MRA4003T3G" H 0   0   50  0001 C CNN "Part number"
@@
 F 0 "C106" H 4732 4104 50  0000 R CNN
 F 1 "10u" H 4732 4195 50  0000 R CNN
-F 2 "" H 4888 4000 50  0001 C CNN
+F 2 "Capacitor_SMD:C_1206_3216Metric_Pad1.42x1.75mm_HandSolder" H 4888 4000 50  0001 C CNN
 F 3 "~" H 4850 4150 50  0001 C CNN
 F 4 "X7R/X5R 25V 1206" H 0   0   50  0001 C CNN "Parameters"
@@
 F 0 "C104" H 4332 4104 50  0000 R CNN
 F 1 "10u" H 4332 4195 50  0000 R CNN
-F 2 "" H 4488 4000 50  0001 C CNN
+F 2 "Capacitor_SMD:C_1206_3216Metric_Pad1.42x1.75mm_HandSolder" H 4488 4000 50  0001 C CNN
 F 3 "~" H 4450 4150 50  0001 C CNN
 F 4 "X7R/X5R 25V 1206" H 0   0   50  0001 C CNN "Parameters"
@@
 F 0 "C102" H 2482 4104 50  0000 R CNN
 F 1 "220u" H 2482 4195 50  0000 R CNN
-F 2 "" H 2638 4000 50  0001 C CNN
+F 2 "Capacitor_SMD:CP_Elec_8x10.5" H 2638 4000 50  0001 C CNN
 F 3 "~" H 2600 4150 50  0001 C CNN
-F 4 "EEE1HA221UAP" H 0   0   50  0001 C CNN "Part number"
+F 4 "EEE1EA221UP" H 0   0   50  0001 C CNN "Part number"
 F 5 "SMT Electrolytic 25V" H 0   0   50  0001 C CNN "Parameters"
 	1    2600 4150
@@
 F 0 "D104" V 3750 4100 50  0000 L CNN
 F 1 "D" V 3650 4100 50  0000 L CNN
-F 2 "" H 4050 4150 50  0001 C CNN
+F 2 "Diode_SMD:D_SOT-23_ANK" H 4050 4150 50  0001 C CNN
 F 3 "~" H 4050 4150 50  0001 C CNN
 F 4 "BAS20" H 0   0   50  0001 C CNN "Part number"
@@
 F 0 "D102" H 2250 3734 50  0000 C CNN
 F 1 "D" H 2250 3825 50  0000 C CNN
-F 2 "" H 2250 3950 50  0001 C CNN
+F 2 "Diode_SMD:D_SMA" H 2250 3950 50  0001 C CNN
 F 3 "~" H 2250 3950 50  0001 C CNN
 F 4 "MRA4003T3G" H 0   0   50  0001 C CNN "Part number"
@@
 F 0 "H101" H 2650 6046 50  0000 L CNN
 F 1 "MountingHole" H 2650 5955 50  0000 L CNN
-F 2 "" H 2550 6000 50  0001 C CNN
+F 2 "MountingHole:MountingHole_2.7mm_M2.5" H 2550 6000 50  0001 C CNN
 F 3 "~" H 2550 6000 50  0001 C CNN
 	1    2550 6000
@@
 F 0 "H103" H 3500 6046 50  0000 L CNN
 F 1 "MountingHole" H 3500 5955 50  0000 L CNN
-F 2 "" H 3400 6000 50  0001 C CNN
+F 2 "MountingHole:MountingHole_2.7mm_M2.5" H 3400 6000 50  0001 C CNN
 F 3 "~" H 3400 6000 50  0001 C CNN
 	1    3400 6000
@@
 F 0 "H102" H 2650 6346 50  0000 L CNN
 F 1 "MountingHole" H 2650 6255 50  0000 L CNN
-F 2 "" H 2550 6300 50  0001 C CNN
+F 2 "MountingHole:MountingHole_2.7mm_M2.5" H 2550 6300 50  0001 C CNN
 F 3 "~" H 2550 6300 50  0001 C CNN
 	1    2550 6300
@@
 F 0 "H104" H 3500 6346 50  0000 L CNN
 F 1 "MountingHole" H 3500 6255 50  0000 L CNN
-F 2 "" H 3400 6300 50  0001 C CNN
+F 2 "MountingHole:MountingHole_2.7mm_M2.5" H 3400 6300 50  0001 C CNN
 F 3 "~" H 3400 6300 50  0001 C CNN
 	1    3400 6300

Commit message: WIP: Assign footprints
Parts:
- R101, R102, R103, R104: footprint (none) -> Resistor_SMD:R_0603_1608Metric_Pad1.05x0.95mm_HandSolder
Changed lines of the file:
@@
 F 0 "R103" H 3700 2400 50  0000 L CNN
 F 1 "240 1%" H 3700 2300 50  0000 L CNN
-F 2 "" V 3730 2700 50  0001 C CNN
+F 2 "Resistor_SMD:R_0603_1608Metric_Pad1.05x0.95mm_HandSolder" V 3730 2700 50  0001 C CNN
 F 3 "~" H 3800 2700 50  0001 C CNN
 F 4 "ERA3AEB241V" H 0   0   50  0001 C CNN "Part number"
@@
 F 0 "R101" H 3400 3100 50  0000 L CNN
 F 1 "3400 1%" H 3400 3000 50  0000 L CNN
-F 2 "" V 3280 3100 50  0001 C CNN
+F 2 "Resistor_SMD:R_0603_1608Metric_Pad1.05x0.95mm_HandSolder" V 3280 3100 50  0001 C CNN
 F 3 "~" H 3350 3100 50  0001 C CNN
 F 4 "MCWF06R3401BTL" H 0   0   50  0001 C CNN "Part number"
@@
 F 0 "R104" H 3700 3850 50  0000 L CNN
 F 1 "240 1%" H 3700 3750 50  0000 L CNN
-F 2 "" V 3730 4150 50  0001 C CNN
+F 2 "Resistor_SMD:R_0603_1608Metric_Pad1.05x0.95mm_HandSolder" V 3730 4150 50  0001 C CNN
 F 3 "~" H 3800 4150 50  0001 C CNN
 F 4 "ERA3AEB241V" H 0   0   50  0001 C CNN "Part number"
@@
 F 0 "R102" H 3400 4550 50  0000 L CNN
 F 1 "3400 1%" H 3400 4450 50  0000 L CNN
-F 2 "" V 3280 4550 50  0001 C CNN
+F 2 "Resistor_SMD:R_0603_1608Metric_Pad1.05x0.95mm_HandSolder" V 3280 4550 50  0001 C CNN
 F 3 "~" H 3350 4550 50  0001 C CNN
 F 4 "MCWF06R3401BTL" H 0   0   50  0001 C CNN "Part number"
