File: actidamp-mk4-smd.sch (KiCad schematic (older format))
At the start: 28 parts, among them J101 XLR3, J102 Phono_Ground, J103 PHONO_IN_L, J104 PHONO_IN_R, J105 LINE_OUT_L, J106 LINE_OUT_R, U101 LM317_3PinPackage, U102 LM337_TO252

Commit message: WIP: Assigning footprints
Parts:
- HS101, HS102: footprint (none) -> actidamp-mk4-smd:Heatsink_TO252_573100
- J103, J104, J105, J106: footprint (none) -> actidamp-mk4-smd:RCA_x1_PJRAN1X1U
- U101, U102: footprint Package_TO_SOT_SMD:TO-252-2 -> Package_TO_SOT_SMD:TO-252-3_TabPin2
Connections:
- wire segments 92 -> 90
- no-connect marks 0 -> 2
Changed lines of the file:
@@
 U 1 1 5D8D1D2C
 P 7050 4050
-F 0 "J103" H 7105 4367 50  0000 C CNN
-F 1 "PHONO_IN_L" H 7105 4276 50  0000 C CNN
-F 2 "" H 7100 4010 50  0001 C CNN
+F 0 "J103" H 6950 5000 50  0000 C CNN
+F 1 "PHONO_IN_L" H 7100 3850 50  0000 C CNN
+F 2 "actidamp-mk4-smd:RCA_x1_PJRAN1X1U" H 7100 4010 50  0001 C CNN
 F 3 "~" H 7100 4010 50  0001 C CNN
 F 4 "PJRAN1X1U02AUX" H 7050 4050 50  0001 C CNN "Part number"
 	1    7050 4050
-	1    0    0    -1
+	1    0    0    1
 $EndComp
 $Comp
@@
 U 1 1 5D8D7FFB
 P 7050 4650
-F 0 "J104" H 7050 5000 50  0000 C CNN
-F 1 "PHONO_IN_R" H 7100 4900 50  0000 C CNN
-F 2 "" H 7100 4610 50  0001 C CNN
+F 0 "J104" H 6950 5550 50  0000 C CNN
+F 1 "PHONO_IN_R" H 7050 4400 50  0000 C CNN
+F 2 "actidamp-mk4-smd:RCA_x1_PJRAN1X1U" H 7100 4610 50  0001 C CNN
 F 3 "~" H 7100 4610 50  0001 C CNN
 F 4 "PJRAN1X1U03AUX" H 2850 1350 50  0001 C CNN "Part number"
 	1    7050 4650
-	1    0    0    1
+	1    0    0    -1
 $EndComp
 $Comp
@@
 	0    -1   -1   0
 $EndComp
-Connection ~ 7350 4150
-Wire Wire Line
-	7350 4150 7350 4050
-Wire Wire Line
-	7350 4650 7350 4550
-Connection ~ 7350 4550
 $Comp
 L Connector:Barrel_Jack_Switch J105
 U 1 1 5D8D8A65
 P 9900 4050
-F 0 "J105" H 9955 4367 50  0000 C CNN
-F 1 "LINE_OUT_L" H 9955 4276 50  0000 C CNN
-F 2 "" H 9950 4010 50  0001 C CNN
+F 0 "J105" H 10000 3850 50  0000 C CNN
+F 1 "LINE_OUT_L" H 9900 3750 50  0000 C CNN
+F 2 "actidamp-mk4-smd:RCA_x1_PJRAN1X1U" H 9950 4010 50  0001 C CNN
 F 3 "~" H 9950 4010 50  0001 C CNN
 F 4 "PJRAN1X1U02AUX" H 3550 1150 50  0001 C CNN "Part number"
 	1    9900 4050
-	-1   0    0    -1
+	-1   0    0    1
 $EndComp
 $Comp
@@
 U 1 1 5D8D8A6B
 P 9900 4450
-F 0 "J106" H 9950 4800 50  0000 C CNN
-F 1 "LINE_OUT_R" H 9950 4700 50  0000 C CNN
-F 2 "" H 9950 4410 50  0001 C CNN
+F 0 "J106" H 10000 4150 50  0000 C CNN
+F 1 "LINE_OUT_R" H 9900 4250 50  0000 C CNN
+F 2 "actidamp-mk4-smd:RCA_x1_PJRAN1X1U" H 9950 4410 50  0001 C CNN
 F 3 "~" H 9950 4410 50  0001 C CNN
 F 4 "PJRAN1X1U03AUX" H 3550 1150 50  0001 C CNN "Part number"
 	1    9900 4450
-	-1   0    0    1
+	-1   0    0    -1
 $EndComp
 $Comp
@@
 Wire Wire Line
 	9500 4250 9600 4250
-Wire Wire Line
-	9600 4250 9600 4150
 Connection ~ 9600 4250
 Wire Wire Line
-	9600 4350 9600 4250
-Wire Wire Line
 	9600 4550 9350 4550
 Wire Wire Line
 	9600 3950 9350 3950
-Wire Wire Line
-	9600 4450 9600 4350
-Connection ~ 9600 4350
-Wire Wire Line
-	9600 4150 9600 4050
-Connection ~ 9600 4150
 $Comp
 L Connector:Screw_Terminal_01x01 J102
@@
 	6500 2650 7750 2650
 Wire Wire Line
-	8100 2650 8100 3800
-Wire Wire Line
 	8100 3800 8300 3800
 $Sheet
@@
 $EndSheet
 Wire Wire Line
-	7350 4150 7350 4350
-Wire Wire Line
 	7450 4350 7350 4350
 Connection ~ 7350 4350
-Wire Wire Line
-	7350 4350 7350 4550
 Wire Wire Line
 	7350 4350 7200 4350
@@
 F 0 "U101" H 3350 2742 50  0000 C CNN
 F 1 "LM317_3PinPackage" H 3350 2651 50  0000 C CNN
-F 2 "Package_TO_SOT_SMD:TO-252-2" H 3350 2750 50  0001 C CIN
+F 2 "Package_TO_SOT_SMD:TO-252-3_TabPin2" H 3350 2750 50  0001 C CIN
 F 3 "http://www.ti.com/lit/ds/symlink/lm317.pdf" H 3350 2500 50  0001 C CNN
 F 4 "" H 0   0   50  0001 C CNN "Additional"
@@
 F 0 "U102" H 3350 3708 50  0000 C CNN
 F 1 "LM337_TO252" H 3350 3799 50  0000 C CNN
-F 2 "Package_TO_SOT_SMD:TO-252-2" H 3350 3750 50  0001 C CIN
+F 2 "Package_TO_SOT_SMD:TO-252-3_TabPin2" H 3350 3750 50  0001 C CIN
 F 3 "http://www.farnell.com/datasheets/1636957.pdf" H 3350 3950 50  0001 C CNN
 F 4 "LM337KVURG3" H 0   0   50  0001 C CNN "Part number"
@@
 F 0 "HS102" H 3941 2291 50  0000 L CNN
 F 1 "Heatsink_Pad" H 3941 2200 50  0000 L CNN
-F 2 "" H 3812 2200 50  0001 C CNN
+F 2 "actidamp-mk4-smd:Heatsink_TO252_573100" H 3812 2200 50  0001 C CNN
 F 3 "~" H 3812 2200 50  0001 C CNN
 F 4 "FK 244 13 D PAK" H 3800 2250 50  0001 C CNN "Part number"
@@
 F 0 "HS101" H 2741 3691 50  0000 L CNN
 F 1 "Heatsink_Pad" H 2741 3600 50  0000 L CNN
-F 2 "" H 2612 3600 50  0001 C CNN
+F 2 "actidamp-mk4-smd:Heatsink_TO252_573100" H 2612 3600 50  0001 C CNN
 F 3 "~" H 2612 3600 50  0001 C CNN
 F 4 "FK 244 13 D PAK" H 2600 3650 50  0001 C CNN "Part number"
@@
 Text Notes 1300 4000 1    50   ~ 0
 Input in range of +-25 up to +-35V
+Wire Wire Line
+	8100 2650 8100 3800
+Wire Wire Line
+	7350 4050 7350 4150
+Wire Wire Line
+	7350 4350 7350 4550
+Wire Wire Line
+	7350 4550 7350 4650
+Connection ~ 7350 4550
+Wire Wire Line
+	7350 4350 7350 4150
+Connection ~ 7350 4150
+Wire Wire Line
+	9600 4250 9600 4350
+Wire Wire Line
+	9600 4250 9600 4150
+NoConn ~ 9600 4050
+NoConn ~ 9600 4450
 $EndSCHEMATC

Commit message: Finish footprints
Parts:
- D101, D102: value D -> MRA4003T3G
- D103, D104: value D -> BAS20
- J101: footprint (none) -> actidamp-mk4-smd:MiniXLR_TRAPC3M1X
- J102: footprint (none) -> actidamp-mk4-smd:SCREW_TERMINAL_SCTM4RA
Changed lines of the file:
@@
 F 0 "J102" H 7400 4250 50  0000 C CNN
 F 1 "Phono_Ground" H 7400 4350 50  0000 C CNN
-F 2 "" H 7000 4350 50  0001 C CNN
+F 2 "actidamp-mk4-smd:SCREW_TERMINAL_SCTM4RA" H 7000 4350 50  0001 C CNN
 F 3 "~" H 7000 4350 50  0001 C CNN
 F 4 "SCRTM4RA" H 7000 4350 50  0001 C CNN "Part number"
@@
 P 4050 2700
 F 0 "D103" V 4350 2650 50  0000 L CNN
-F 1 "D" V 4450 2650 50  0000 L CNN
+F 1 "BAS20" V 4450 2650 50  0000 L CNN
 F 2 "Diode_SMD:D_SOT-23_ANK" H 4050 2700 50  0001 C CNN
 F 3 "~" H 4050 2700 50  0001 C CNN
@@
 P 2250 2500
 F 0 "D101" H 2250 2284 50  0000 C CNN
-F 1 "D" H 2250 2375 50  0000 C CNN
+F 1 "MRA4003T3G" H 2250 2375 50  0000 C CNN
 F 2 "Diode_SMD:D_SMA" H 2250 2500 50  0001 C CNN
 F 3 "~" H 2250 2500 50  0001 C CNN
@@
 P 4050 4150
 F 0 "D104" V 3750 4100 50  0000 L CNN
-F 1 "D" V 3650 4100 50  0000 L CNN
+F 1 "BAS20" V 3650 4100 50  0000 L CNN
 F 2 "Diode_SMD:D_SOT-23_ANK" H 4050 4150 50  0001 C CNN
 F 3 "~" H 4050 4150 50  0001 C CNN
@@
 P 2250 3950
 F 0 "D102" H 2250 3734 50  0000 C CNN
-F 1 "D" H 2250 3825 50  0000 C CNN
+F 1 "MRA4003T3G" H 2250 3825 50  0000 C CNN
 F 2 "Diode_SMD:D_SMA" H 2250 3950 50  0001 C CNN
 F 3 "~" H 2250 3950 50  0001 C CNN
@@
 F 0 "J101" V 1846 3478 50  0000 L CNN
 F 1 "XLR3" V 1755 3478 50  0000 L CNN
-F 2 "" H 1800 3250 50  0001 C CNN
+F 2 "actidamp-mk4-smd:MiniXLR_TRAPC3M1X" H 1800 3250 50  0001 C CNN
 F 3 " ~" H 1800 3250 50  0001 C CNN
 F 4 "TRAPC3MX" H 600 0   50  0001 C CNN "Part number"

Commit message: More routing
Parts:
- removed H101, H102, H103, H104: MountingHole, MountingHole:MountingHole_2.7mm_M2.5, symbol Mechanical:MountingHole
Changed lines of the file:
@@
 EESchema Schematic File Version 4
 LIBS:actidamp-mk4-smd-cache
-EELAYER 26 0
+EELAYER 30 0
 EELAYER END
 $Descr A4 11693 8268
@@
 	2150 3250 2100 3250
 $Comp
-L Mechanical:MountingHole H101
-U 1 1 5D6E3F66
-P 2550 6000
-F 0 "H101" H 2650 6046 50  0000 L CNN
-F 1 "MountingHole" H 2650 5955 50  0000 L CNN
-F 2 "MountingHole:MountingHole_2.7mm_M2.5" H 2550 6000 50  0001 C CNN
-F 3 "~" H 2550 6000 50  0001 C CNN
-	1    2550 6000
-	1    0    0    -1
-$EndComp
-$Comp
-L Mechanical:MountingHole H103
-U 1 1 5D6E3FDD
-P 3400 6000
-F 0 "H103" H 3500 6046 50  0000 L CNN
-F 1 "MountingHole" H 3500 5955 50  0000 L CNN
-F 2 "MountingHole:MountingHole_2.7mm_M2.5" H 3400 6000 50  0001 C CNN
-F 3 "~" H 3400 6000 50  0001 C CNN
-	1    3400 6000
-	1    0    0    -1
-$EndComp
-$Comp
-L Mechanical:MountingHole H102
-U 1 1 5D6E4023
-P 2550 6300
-F 0 "H102" H 2650 6346 50  0000 L CNN
-F 1 "MountingHole" H 2650 6255 50  0000 L CNN
-F 2 "MountingHole:MountingHole_2.7mm_M2.5" H 2550 6300 50  0001 C CNN
-F 3 "~" H 2550 6300 50  0001 C CNN
-	1    2550 6300
-	1    0    0    -1
-$EndComp
-$Comp
-L Mechanical:MountingHole H104
-U 1 1 5D6E406B
-P 3400 6300
-F 0 "H104" H 3500 6346 50  0000 L CNN
-F 1 "MountingHole" H 3500 6255 50  0000 L CNN
-F 2 "MountingHole:MountingHole_2.7mm_M2.5" H 3400 6300 50  0001 C CNN
-F 3 "~" H 3400 6300 50  0001 C CNN
-	1    3400 6300
-	1    0    0    -1
-$EndComp
-$Comp
 L Mechanical:Heatsink_Pad HS102
