File: channel.sch (KiCad schematic (older format))
At the start: 35 parts

Commit message: Capture of original actidamp iv
Parts:
- removed C?: C, symbol Device:C
- removed R?: R, symbol Device:R
- added C? (x17): C, symbol Device:C
- added J?: Conn_01x03, symbol Connector_Generic:Conn_01x03
- added R? (x16): R, symbol Device:R
- added RV?: R_POT_TRIM, symbol Device:R_POT_TRIM
- added U? (x2): NE5534, symbol Amplifier_Operational:NE5534
- added U?: LF411, symbol actidamp:LF411
Connections:
- net labels added: +19, -19, IN, OUT
- wire segments 91 -> 224

Commit message: Assign capacitors, redo hierarchy
Parts:
- removed C? (x5): C, symbol Device:C
- removed J?: Conn_01x03, symbol Connector_Generic:Conn_01x03
- removed Q? (x2): Q_NJFET_DGS, symbol Device:Q_NJFET_DGS
- removed R? (x4): R, symbol Device:R
- removed U? (x4): NE5534, symbol Amplifier_Operational:NE5534
- added C13, C15, C16: 470n, symbol Device:C
- added C18, C19, C20: 100n, symbol Device:C
- added C30, C31: 2.7n, symbol Device:C
- added C32: 1.5n, symbol Device:C
- added Q1: 2SK3320, symbol actidamp:Q_DUAL_N_JFET
- added R13: 12k, symbol Device:R
- added R17: 4k7, symbol Device:R
- added R19: 82k, symbol Device:R
- added SW2: SW_SP3T, symbol Switch:SW_SP3T
- added U2, U4: NE5532, symbol Amplifier_Operational:NE5532
- C1, C14, C8: renamed from C?; value C -> 100p; Part number (none) -> 06035A101JAT2A
- C10, C11: renamed from C?; value C -> 1u; Part number (none) -> SMDIC04100TB00KQ00
- C12: renamed from C?; value C -> 680p; Part number (none) -> SMDIC03680TB00KQ00
- C17, C26, C29: renamed from C?; value C -> 680n; Part number (none) -> SMDIC03680TB00KQ00
- C2: renamed from C?; value C -> 220p; Part number (none) -> 06035A221JAT2A
- C21, C22, C23: renamed from C?; value C -> 100n; Part number (none) -> ECHU1H104GX9
- C24: renamed from C?; value C -> 220p; Part number (none) -> ECHU1H221GX5
- C25, C27, C28: renamed from C?; value C -> 2.7n; Part number (none) -> ECHU1H272GX5
- C3: renamed from C?; value C -> 330p; Part number (none) -> 06035A331JAT2A
- C4, C7: renamed from C?; value C -> 470p; Part number (none) -> 06035A471JAT2A
- C5, C6: renamed from C?; value C -> 15p; Part number (none) -> 06035A150JAT2A
- C9: renamed from C?; value C -> 10p; Part number (none) -> 06035A100JAT2A
- L1: renamed from L?; value L -> 220uH
- R1: renamed from R?; value R -> 220
- R10: renamed from R?; value R -> 5k1
- R11, R4: renamed from R?; value R -> 1M6
- R12, R29: renamed from R?; value R -> 100
- R14, R24, R8: renamed from R?; value R -> 3k3
- R15, R18: renamed from R?; value R -> 12k
- R16, R26: renamed from R?; value R -> 1M
- R2: renamed from R?; value R -> 51k
- R20: renamed from R?; value R -> 4770 1%
- R21: renamed from R?; value R -> 530 1%
- R22: renamed from R?; value R -> 390
- R23: renamed from R?; value R -> 6k8
- R25: renamed from R?; value R -> 5k 1%
- R27: renamed from R?; value R -> 1k
- R28: renamed from R?; value R -> 750
- R3: renamed from R?; value R -> 47
- R5, R7: renamed from R?; value R -> 1k8
- R6, R9: renamed from R?; value R -> 10k
- RV1: renamed from RV?; value R_POT_TRIM -> 10k
- SW1: renamed from SW?; Part number (none) -> 1571983-5
- U1: renamed from U?; Part number (none) -> NE5534DG
- U3, U5: renamed from U?; Part number (none) -> LF411CD
Connections:
- net labels added: V+, V-
- net labels removed: +19, -19
- wire segments 224 -> 223

Commit message: All schematics drafted
Parts:
- L1: Part number (none) -> NLFV32T-221K-EF
- Q1: Part number (none) -> 2SK3320
Changed lines of the file:
@@
 $Descr A4 11693 8268
 encoding utf-8
-Sheet 2 3
+Sheet 2 5
 Title ""
 Date ""
@@
 F 2 "" H 1850 3150 50  0001 C CNN
 F 3 "~" H 1850 3150 50  0001 C CNN
+F 4 "NLFV32T-221K-EF" V 1850 3150 50  0001 C CNN "Part number"
 	1    1850 3150
 	0    -1   -1   0
@@
 F 2 "" H 3000 3550 50  0001 C CNN
 F 3 "~" H 2800 3450 50  0001 C CNN
+F 4 "2SK3320" H 0   0   50  0001 C CNN "Part number"
 	1    2800 3450
 	1    0    0    -1
@@
 F 2 "" H 3700 3550 50  0001 C CNN
 F 3 "~" H 3500 3450 50  0001 C CNN
+F 4 "2SK3320" H 0   0   50  0001 C CNN "Part number"
 	2    3500 3450
 	-1   0    0    -1
@@
 F 1 "SW_SP3T" H 5750 2700 50  0000 C CNN
 F 2 "" H 5125 3125 50  0001 C CNN
-F 3 "~" H 5125 3125 50  0001 C CNN
+F 3 "http://www.farnell.com/datasheets/2604289.pdf" H 5125 3125 50  0001 C CNN
 F 4 "CL-SB-13B-02T" H 0   0   50  0001 C CNN "Part number"
 	1    5750 2950

Commit message: Finalise schematics with power supplies and successful ERC
Parts:
- renumbered C1 to C201, C2 to C202, C3 to C203, C4 to C204, C5 to C205, C6 to C206, C7 to C207, C8 to C208, C9 to C209, C10 to C210, C11 to C211, C12 to C212, C13 to C213, C14 to C214, C15 to C215, C16 to C216, C17 to C217, C18 to C218, C19 to C219, C20 to C220, C21 to C221, C22 to C222, C23 to C223, C24 to C224, C25 to C225, C26 to C226, C27 to C227, C28 to C228, C29 to C229, C30 to C230, C31 to C231, C32 to C232, L1 to L201, Q1 to Q201, R1 to R201, R2 to R202, R3 to R203, R4 to R204, R5 to R205, R6 to R206, R7 to R207, R8 to R208, R9 to R209, R10 to R210, R11 to R211, R12 to R212, R13 to R213, R14 to R214, R15 to R215, R16 to R216, R17 to R217, R18 to R218, R19 to R219, R20 to R220, R21 to R221, R22 to R222, R23 to R223, R24 to R224, R25 to R225, R26 to R226, R27 to R227, R28 to R228, R29 to R229, RV1 to RV201, SW1 to SW201, SW2 to SW202, U1 to U201, U2 to U202, U3 to U203, U4 to U204, U5 to U205
Connections:
- wire segments 223 -> 224
- no-connect marks 0 -> 4

Commit message: Finalise BOM
Parts:
- C201, C202, C203, C204, C205, C206, C207, C208, C209, C212, C213, C214, C215, C216, C217, C224, C226, C229: Parameters (none) -> X7R/X5R 0603
- C210, C211: Parameters (none) -> X7R/X5R 25V 0603
- C218, C219, C220: Parameters (none) -> PPS 1913
- C221, C222: value 100n -> 120n; Parameters (none) -> PPS 2416; Part number ECHU1H104GX9 -> ECHU1H124GX9
- C223: value 100n -> 47n; Parameters (none) -> PPS 1913; Part number ECHU1H104GX9 -> ECHU1H473GX9
- C225, C227, C228, C230, C231, C232: Parameters (none) -> PPS 0805
- R201: Parameters (none) -> Thin Film 0603; Part number (none) -> ERA3AEB221V
- R202: Parameters (none) -> Thin Film 0603; Part number (none) -> ERA3AEB513V
- R203: Parameters (none) -> Thin Film 0603; Part number (none) -> RT0603FRE0747RL
- R204, R211: Parameters (none) -> Thin Film 0805; Part number (none) -> 1-1614959-2
- R205, R207: value 1k8 -> 1k8 1/8W; Parameters (none) -> Thin Film 0805; Part number (none) -> RT0805FRE071K8L
- R206, R209: value 10k -> 10k 1%; Parameters (none) -> Thin Film 0603; Part number (none) -> RT0603WRE0710KL
- R208: value 3k3 -> 3k3 1/4W; Parameters (none) -> Thin Film 1206; Part number (none) -> ERA8ARB332V
- R210: Parameters (none) -> Thin Film 0603; Part number (none) -> ERA3AEB512V
- R212: value 100 -> 100 1%; Parameters (none) -> Thin Film 0603; Part number (none) -> RT0603FRE07100RL
- R213, R215, R218: Parameters (none) -> Thin Film 0603; Part number (none) -> ERA3AEB123V
- R214: value 3k3 -> 3k3 1%; Parameters (none) -> Thin Film 0603; Part number (none) -> RT0603FRE073K3L
- R216, R226: Parameters (none) -> Thin Film 0603; Part number (none) -> MCT06030C1004FP500
- R217: Parameters (none) -> Thin Film 0603; Part number (none) -> RT0603FRE074K7L
- R219: Parameters (none) -> Thin Film 0603; Part number (none) -> ERA3AEB823V
- R220: value 4770 1% -> 4k87 1%; Parameters (none) -> Thin Film 0603; Part number (none) -> CPF0603F4K87C1
- R221: value 530 1% -> 542 1%; Parameters (none) -> Thin Film 0603; Part number (none) -> RN73H1JTTD5420B50
- R222: value 390 -> 390 1%; Parameters (none) -> Thin Film 0603; Part number (none) -> RT0603FRE07390RL
- R223: value 6k8 -> 6k8 1%; Parameters (none) -> Thin Film 0603; Part number (none) -> RT0603FRE076K8L
- R224: Parameters (none) -> Thin Film 0603; Part number (none) -> RT0603FRE073K3L
- R225: Parameters (none) -> Thin Film 0603; Part number (none) -> RT0603BRE075KL
- R227: Parameters (none) -> Thin Film 0603; Part number (none) -> RT0603FRE071KL
- R228: Parameters (none) -> Thin Film 0603; Part number (none) -> MCT06030C7500FP500
- R229: Parameters (none) -> Thin Film 0603; Part number (none) -> MCT06030C1000FP500
Other:
- note added: "All resistors are metal film"

Commit message: WIP: Assign footprints
Parts:
- C201, C208, C214: footprint (none) -> Capacitor_SMD:C_0603_1608Metric_Pad1.05x0.95mm_HandSolder; Parameters X7R/X5R 0603 -> C0G 0603; Part number 06035A101JAT2A -> MC0603N101J500CT
- C202: footprint (none) -> Capacitor_SMD:C_0603_1608Metric_Pad1.05x0.95mm_HandSolder; Parameters X7R/X5R 0603 -> C0G 0603
- C203: footprint (none) -> Capacitor_SMD:C_0603_1608Metric_Pad1.05x0.95mm_HandSolder; Parameters X7R/X5R 0603 -> C0G 0603; Part number 06035A331JAT2A -> MC0603N331J500CT
- C204, C207: footprint (none) -> Capacitor_SMD:C_0603_1608Metric_Pad1.05x0.95mm_HandSolder; Parameters X7R/X5R 0603 -> C0G 0603; Part number 06035A471JAT2A -> VJ0603A471JXACW1BC
- C205, C206: footprint (none) -> Capacitor_SMD:C_0603_1608Metric_Pad1.05x0.95mm_HandSolder; Parameters X7R/X5R 0603 -> C0G 0603; Part number 06035A150JAT2A -> MC0603N150J500CT
- C209: footprint (none) -> Capacitor_SMD:C_0603_1608Metric_Pad1.05x0.95mm_HandSolder; Parameters X7R/X5R 0603 -> C0G 0603; Part number 06035A100JAT2A -> MC0603N100J500CT
- C210, C211: Parameters X7R/X5R 25V 0603 -> PPS 2824
- C212: value 680p -> 680n; Parameters X7R/X5R 0603 -> PPS 2824
- C213, C215, C216, C217, C226, C229: Parameters X7R/X5R 0603 -> PPS 2824
- C224: footprint (none) -> Capacitor_SMD:C_0805_2012Metric_Pad1.15x1.40mm_HandSolder; Parameters X7R/X5R 0603 -> PPS 0805
- C225, C227, C228, C230, C231, C232: footprint (none) -> Capacitor_SMD:C_0805_2012Metric_Pad1.15x1.40mm_HandSolder
- U201, U202, U203, U204, U205: footprint (none) -> Package_SO:SOIC-8-1EP_3.9x4.9mm_P1.27mm_EP2.29x3mm

Commit message: WIP: Assign footprints
Parts:
- R201, R202, R203, R206, R209, R210, R212, R213, R214, R215, R216, R217, R218, R219, R220, R221, R222, R223, R224, R225, R226, R227, R228, R229: footprint (none) -> Resistor_SMD:R_0603_1608Metric_Pad1.05x0.95mm_HandSolder
- R204, R205, R207, R211: footprint (none) -> Resistor_SMD:R_0805_2012Metric_Pad1.15x1.40mm_HandSolder
- R208: footprint (none) -> Resistor_SMD:R_1206_3216Metric_Pad1.42x1.75mm_HandSolder
- RV201: footprint (none) -> Potentiometer_SMD:Potentiometer_Vishay_TS53YJ_Vertical; Part number (none) -> TS53YJ103MR10

Commit message: WIP: Assigning footprints
Parts:
- removed SW202: SW_SP3T, symbol Switch:SW_SP3T
- removed U201: NE5534, Package_SO:SOIC-8-1EP_3.9x4.9mm_P1.27mm_EP2.29x3mm, symbol Amplifier_Operational:NE5534
- removed unit 2 of U202
- added R230: 1M, Resistor_SMD:R_0603_1608Metric_Pad1.05x0.95mm_HandSolder, symbol Device:R
- added SW202: SW_DPDT_x2, actidamp-mk4-smd:Wurth_452403012014, symbol Switch:SW_DPDT_x2
- added unit 1 of U201
- added U202: NE5534, Package_SO:SOIC-8_3.9x4.9mm_P1.27mm, symbol Amplifier_Operational:NE5534
- C209: Part number MC0603N100J500CT -> MC0603N100J500CT
- C210, C211, C212, C213, C215, C216, C217, C226, C229: footprint (none) -> actidamp-mk4-smd:C_2824_7260Metric_Pad3.20x4.45mm_HandSolder
- C218, C219, C220, C223: footprint (none) -> actidamp-mk4-smd:C_1913_4833Metric_Pad1.3x3.00mm_HandSolder
- C221, C222: footprint (none) -> actidamp-mk4-smd:C_2416_6041Metric_Pad1.5x3.8mm_HandSolder
- C224, C225, C227, C228, C230, C231, C232: footprint Capacitor_SMD:C_0805_2012Metric_Pad1.15x1.40mm_HandSolder -> actidamp-mk4-smd:C_0805_2012Metric_Pad1.15x1.1mm_HandSolder
- SW201: footprint (none) -> actidamp-mk4-smd:SW_DIP_SPSTx04_Slide_TE_1571983-5_W6.2mm_P1.27mm
- U201: renamed from U202; footprint Package_SO:SOIC-8-1EP_3.9x4.9mm_P1.27mm_EP2.29x3mm -> Package_SO:SOIC-8_3.9x4.9mm_P1.27mm
- U203, U204, U205: footprint Package_SO:SOIC-8-1EP_3.9x4.9mm_P1.27mm_EP2.29x3mm -> Package_SO:SOIC-8_3.9x4.9mm_P1.27mm
Connections:
- wire segments 224 -> 229
- no-connect marks 4 -> 2
Other:
- note added: "All resistors are thin film / metal film"
- note removed: "All resistors are metal film"
