File: channel.sch (KiCad schematic (older format))
At the start: 72 parts, among them Q201 2SK3320, SW201 SW_DIP_x04, SW202 SW_DPDT_x2, U201 NE5532, U202 NE5534, U203 LF411, U204 NE5532, U205 LF411

Commit message: Finish footprints
Parts:
- L201: footprint (none) -> actidamp-mk4-smd:L_NLFV32_Pad1.2x2.0mm_HandSolder
- Q201: footprint (none) -> Package_TO_SOT_SMD:SOT-353_SC-70-5_Handsoldering
Changed lines of the file:
@@
 AR Path="/5C72F90C/5C7337D1" Ref="#PWR0201"  Part="1"
 AR Path="/5C7379E1/5C7337D1" Ref="#PWR0301"  Part="1"
-F 0 "#PWR0301" H 1150 4600 50  0001 C CNN
+F 0 "#PWR0201" H 1150 4600 50  0001 C CNN
 F 1 "GND" H 1155 4677 50  0000 C CNN
 F 2 "" H 1150 4850 50  0001 C CNN
@@
 AR Path="/5C72F90C/5C7337D7" Ref="#PWR0202"  Part="1"
 AR Path="/5C7379E1/5C7337D7" Ref="#PWR0302"  Part="1"
-F 0 "#PWR0302" H 1350 4600 50  0001 C CNN
+F 0 "#PWR0202" H 1350 4600 50  0001 C CNN
 F 1 "GND" H 1355 4677 50  0000 C CNN
 F 2 "" H 1350 4850 50  0001 C CNN
@@
 AR Path="/5C72F90C/5C7337DD" Ref="#PWR0203"  Part="1"
 AR Path="/5C7379E1/5C7337DD" Ref="#PWR0303"  Part="1"
-F 0 "#PWR0303" H 1550 4600 50  0001 C CNN
+F 0 "#PWR0203" H 1550 4600 50  0001 C CNN
 F 1 "GND" H 1555 4677 50  0000 C CNN
 F 2 "" H 1550 4850 50  0001 C CNN
@@
 AR Path="/5C72F90C/5C7337E3" Ref="#PWR0204"  Part="1"
 AR Path="/5C7379E1/5C7337E3" Ref="#PWR0304"  Part="1"
-F 0 "#PWR0304" H 1750 4600 50  0001 C CNN
+F 0 "#PWR0204" H 1750 4600 50  0001 C CNN
 F 1 "GND" H 1755 4677 50  0000 C CNN
 F 2 "" H 1750 4850 50  0001 C CNN
@@
 F 0 "L201" V 2040 3150 50  0000 C CNN
 F 1 "220uH" V 1949 3150 50  0000 C CNN
-F 2 "" H 1850 3150 50  0001 C CNN
+F 2 "actidamp-mk4-smd:L_NLFV32_Pad1.2x2.0mm_HandSolder" H 1850 3150 50  0001 C CNN
 F 3 "~" H 1850 3150 50  0001 C CNN
 F 4 "NLFV32T-221K-EF" V 1850 3150 50  0001 C CNN "Part number"
@@
 AR Path="/5C72F90C/5C733829" Ref="#PWR0205"  Part="1"
 AR Path="/5C7379E1/5C733829" Ref="#PWR0305"  Part="1"
-F 0 "#PWR0305" H 2050 4600 50  0001 C CNN
+F 0 "#PWR0205" H 2050 4600 50  0001 C CNN
 F 1 "GND" H 2055 4677 50  0000 C CNN
 F 2 "" H 2050 4850 50  0001 C CNN
@@
 AR Path="/5C72F90C/5C733837" Ref="#PWR0206"  Part="1"
 AR Path="/5C7379E1/5C733837" Ref="#PWR0306"  Part="1"
-F 0 "#PWR0306" H 2350 4600 50  0001 C CNN
+F 0 "#PWR0206" H 2350 4600 50  0001 C CNN
 F 1 "GND" H 2355 4677 50  0000 C CNN
 F 2 "" H 2350 4850 50  0001 C CNN
@@
 AR Path="/5C72F90C/5C7338DB" Ref="#PWR0210"  Part="1"
 AR Path="/5C7379E1/5C7338DB" Ref="#PWR0310"  Part="1"
-F 0 "#PWR0310" H 5000 5100 50  0001 C CNN
+F 0 "#PWR0210" H 5000 5100 50  0001 C CNN
 F 1 "GND" H 5005 5177 50  0000 C CNN
 F 2 "" H 5000 5350 50  0001 C CNN
@@
 AR Path="/5C72F90C/5C73390F" Ref="#PWR0208"  Part="1"
 AR Path="/5C7379E1/5C73390F" Ref="#PWR0308"  Part="1"
-F 0 "#PWR0308" H 4600 3600 50  0001 C CNN
+F 0 "#PWR0208" H 4600 3600 50  0001 C CNN
 F 1 "GND" H 4605 3677 50  0000 C CNN
 F 2 "" H 4600 3850 50  0001 C CNN
@@
 AR Path="/5C72F90C/5C7B8E68" Ref="#PWR0207"  Part="1"
 AR Path="/5C7379E1/5C7B8E68" Ref="#PWR0307"  Part="1"
-F 0 "#PWR0307" H 3850 5150 50  0001 C CNN
+F 0 "#PWR0207" H 3850 5150 50  0001 C CNN
 F 1 "GND" H 3855 5227 50  0000 C CNN
 F 2 "" H 3850 5400 50  0001 C CNN
@@
 AR Path="/5C72F90C/5C8A14EB" Ref="#PWR0213"  Part="1"
 AR Path="/5C7379E1/5C8A14EB" Ref="#PWR0313"  Part="1"
-F 0 "#PWR0313" H 6750 3500 50  0001 C CNN
+F 0 "#PWR0213" H 6750 3500 50  0001 C CNN
 F 1 "GND" H 6755 3577 50  0000 C CNN
 F 2 "" H 6750 3750 50  0001 C CNN
@@
 AR Path="/5C72F90C/5C8A155E" Ref="#PWR0214"  Part="1"
 AR Path="/5C7379E1/5C8A155E" Ref="#PWR0314"  Part="1"
-F 0 "#PWR0314" H 7350 3500 50  0001 C CNN
+F 0 "#PWR0214" H 7350 3500 50  0001 C CNN
 F 1 "GND" H 7355 3577 50  0000 C CNN
 F 2 "" H 7350 3750 50  0001 C CNN
@@
 AR Path="/5C72F90C/5C95B9B2" Ref="#PWR0216"  Part="1"
 AR Path="/5C7379E1/5C95B9B2" Ref="#PWR0316"  Part="1"
-F 0 "#PWR0316" H 8500 3200 50  0001 C CNN
+F 0 "#PWR0216" H 8500 3200 50  0001 C CNN
 F 1 "GND" H 8505 3277 50  0000 C CNN
 F 2 "" H 8500 3450 50  0001 C CNN
@@
 AR Path="/5C72F90C/5C961584" Ref="#PWR0217"  Part="1"
 AR Path="/5C7379E1/5C961584" Ref="#PWR0317"  Part="1"
-F 0 "#PWR0317" H 8700 3200 50  0001 C CNN
+F 0 "#PWR0217" H 8700 3200 50  0001 C CNN
 F 1 "GND" H 8705 3277 50  0000 C CNN
 F 2 "" H 8700 3450 50  0001 C CNN
@@
 AR Path="/5C72F90C/5C961607" Ref="#PWR0218"  Part="1"
 AR Path="/5C7379E1/5C961607" Ref="#PWR0318"  Part="1"
-F 0 "#PWR0318" H 8900 3200 50  0001 C CNN
+F 0 "#PWR0218" H 8900 3200 50  0001 C CNN
 F 1 "GND" H 8905 3277 50  0000 C CNN
 F 2 "" H 8900 3450 50  0001 C CNN
@@
 AR Path="/5C72F90C/5CA61BAB" Ref="#PWR0221"  Part="1"
 AR Path="/5C7379E1/5CA61BAB" Ref="#PWR0321"  Part="1"
-F 0 "#PWR0321" H 9250 4900 50  0001 C CNN
+F 0 "#PWR0221" H 9250 4900 50  0001 C CNN
 F 1 "GND" H 9255 4977 50  0000 C CNN
 F 2 "" H 9250 5150 50  0001 C CNN
@@
 AR Path="/5C72F90C/5CA69810" Ref="#PWR0219"  Part="1"
 AR Path="/5C7379E1/5CA69810" Ref="#PWR0319"  Part="1"
-F 0 "#PWR0319" H 9000 3900 50  0001 C CNN
+F 0 "#PWR0219" H 9000 3900 50  0001 C CNN
 F 1 "GND" H 9005 3977 50  0000 C CNN
 F 2 "" H 9000 4150 50  0001 C CNN
@@
 AR Path="/5C72F90C/5CAB1C95" Ref="#PWR0224"  Part="1"
 AR Path="/5C7379E1/5CAB1C95" Ref="#PWR0324"  Part="1"
-F 0 "#PWR0324" H 9650 3900 50  0001 C CNN
+F 0 "#PWR0224" H 9650 3900 50  0001 C CNN
 F 1 "GND" H 9655 3977 50  0000 C CNN
 F 2 "" H 9650 4150 50  0001 C CNN
@@
 AR Path="/5C72F90C/5D1214D2" Ref="#PWR0209"  Part="1"
 AR Path="/5C7379E1/5D1214D2" Ref="#PWR0309"  Part="1"
-F 0 "#PWR0309" H 4800 2200 50  0001 C CNN
+F 0 "#PWR0209" H 4800 2200 50  0001 C CNN
 F 1 "GND" H 4805 2277 50  0000 C CNN
 F 2 "" H 4800 2450 50  0001 C CNN
@@
 AR Path="/5C72F90C/5D1889AA" Ref="#PWR0212"  Part="1"
 AR Path="/5C7379E1/5D1889AA" Ref="#PWR0312"  Part="1"
-F 0 "#PWR0312" H 5600 2200 50  0001 C CNN
+F 0 "#PWR0212" H 5600 2200 50  0001 C CNN
 F 1 "GND" H 5605 2277 50  0000 C CNN
 F 2 "" H 5600 2450 50  0001 C CNN
@@
 F 0 "Q201" H 2450 3700 50  0000 L CNN
 F 1 "2SK3320" H 2400 3600 50  0000 L CNN
-F 2 "" H 3000 3550 50  0001 C CNN
+F 2 "Package_TO_SOT_SMD:SOT-353_SC-70-5_Handsoldering" H 3000 3550 50  0001 C CNN
 F 3 "~" H 2800 3450 50  0001 C CNN
 F 4 "2SK3320" H 0   0   50  0001 C CNN "Part number"
@@
 F 0 "Q201" H 3150 3700 50  0000 L CNN
 F 1 "2SK3320" H 3100 3600 50  0000 L CNN
-F 2 "" H 3700 3550 50  0001 C CNN
+F 2 "Package_TO_SOT_SMD:SOT-353_SC-70-5_Handsoldering" H 3700 3550 50  0001 C CNN
 F 3 "~" H 3500 3450 50  0001 C CNN
 F 4 "2SK3320" H 0   0   50  0001 C CNN "Part number"
@@
 AR Path="/5C72F90C/5D73C793" Ref="#PWR0220"  Part="1"
 AR Path="/5C7379E1/5D73C793" Ref="#PWR0320"  Part="1"
-F 0 "#PWR0320" H 9100 3200 50  0001 C CNN
+F 0 "#PWR0220" H 9100 3200 50  0001 C CNN
 F 1 "GND" H 9105 3277 50  0000 C CNN
 F 2 "" H 9100 3450 50  0001 C CNN
@@
 AR Path="/5C72F90C/5D73C838" Ref="#PWR0222"  Part="1"
 AR Path="/5C7379E1/5D73C838" Ref="#PWR0322"  Part="1"
-F 0 "#PWR0322" H 9300 3200 50  0001 C CNN
+F 0 "#PWR0222" H 9300 3200 50  0001 C CNN
 F 1 "GND" H 9305 3277 50  0000 C CNN
 F 2 "" H 9300 3450 50  0001 C CNN
@@
 AR Path="/5C72F90C/5D73C8DD" Ref="#PWR0223"  Part="1"
 AR Path="/5C7379E1/5D73C8DD" Ref="#PWR0323"  Part="1"
-F 0 "#PWR0323" H 9500 3200 50  0001 C CNN
+F 0 "#PWR0223" H 9500 3200 50  0001 C CNN
 F 1 "GND" H 9505 3277 50  0000 C CNN
 F 2 "" H 9500 3450 50  0001 C CNN
@@
 AR Path="/5C72F90C/5D75A593" Ref="#PWR0112"  Part="1"
 AR Path="/5C7379E1/5D75A593" Ref="#PWR0113"  Part="1"
-F 0 "#PWR0113" H 5400 4900 50  0001 C CNN
+F 0 "#PWR0112" H 5400 4900 50  0001 C CNN
 F 1 "GND" H 5405 4977 50  0000 C CNN
 F 2 "" H 5400 5150 50  0001 C CNN
@@
 AR Path="/5C72F90C/5D766F0B" Ref="#PWR0114"  Part="1"
 AR Path="/5C7379E1/5D766F0B" Ref="#PWR0115"  Part="1"
-F 0 "#PWR0115" H 7550 3750 50  0001 C CNN
+F 0 "#PWR0114" H 7550 3750 50  0001 C CNN
 F 1 "GND" H 7555 3827 50  0000 C CNN
 F 2 "" H 7550 4000 50  0001 C CNN

Commit message: Routing.. routing.. routing
Connections:
- net at C208.2, R204.2, R206.1: now also U201.7; no longer U201.1
- net at C207.1, Q201.1 (D), R205.2: now also U201.2 (-); no longer U201.6 (-)
- net at Q201.3 (D), R203.1, R207.2: now also U201.3 (+); no longer U201.5 (+)
- net at C208.1, R206.2, R209.1: now also U201.6 (-); no longer U201.2 (-)
- net at C213.2, C214.1, R209.2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: now also SW202.1 (A), U201.1; no longer SW202.3 (C), U201.7
- net at C210.1, R210.1: now also U201.5 (+); no longer U201.3 (+)
- net at R217.1, U202.2 (-), U202.6: now also SW202.3 (C); no longer SW202.1 (A)
Changed lines of the file:
@@
 $Descr A4 11693 8268
 encoding utf-8
-Sheet 3 5
+Sheet 2 5
 Title ""
 Date ""
@@
 $Comp
 L Amplifier_Operational:NE5532 U201
-U 2 1 5CFDF7B0
+U 1 1 5CFDF7B0
 P 3900 2900
-AR Path="/5C72F90C/5CFDF7B0" Ref="U201"  Part="2"
+AR Path="/5C72F90C/5CFDF7B0" Ref="U201"  Part="1"
 AR Path="/5C7379E1/5CFDF7B0" Ref="U301"  Part="1"
 F 0 "U201" H 3900 3267 50  0000 C CNN
@@
 F 3 "http://www.farnell.com/datasheets/2160703.pdf" H 3900 2900 50  0001 C CNN
 F 4 "NE5534ADG" H 0   0   50  0001 C CNN "Part number"
-	2    3900 2900
+	1    3900 2900
 	1    0    0    -1
 $EndComp
@@
 AR Path="/5C72F90C/5D71A7DA" Ref="SW202"  Part="1"
 AR Path="/5C7379E1/5D71A7DA" Ref="SW202"  Part="2"
-F 0 "SW202" H 5700 2650 50  0000 C CNN
-F 1 "SW_DPDT_x2" H 5700 2500 50  0000 C CNN
+F 0 "SW202" H 5700 3450 50  0000 C CNN
+F 1 "SW_DPDT_x2" H 5650 3350 50  0000 C CNN
 F 2 "actidamp-mk4-smd:Wurth_452403012014" H 5750 2950 50  0001 C CNN
 F 3 "~" H 5750 2950 50  0001 C CNN
 F 4 "452403012014" H 0   0   50  0001 C CNN "Part number"
 	1    5750 2950
-	-1   0    0    -1
+	-1   0    0    1
 $EndComp
 $Comp
 L Amplifier_Operational:NE5532 U201
-U 1 1 5D72AFBD
+U 2 1 5D72AFBD
 P 3300 4800
-AR Path="/5C72F90C/5D72AFBD" Ref="U201"  Part="1"
+AR Path="/5C72F90C/5D72AFBD" Ref="U201"  Part="2"
 AR Path="/5C7379E1/5D72AFBD" Ref="U301"  Part="2"
 F 0 "U201" H 3300 5167 50  0000 C CNN
@@
 F 3 "http://www.farnell.com/datasheets/2160703.pdf" H 3300 4800 50  0001 C CNN
 F 4 "NE5534ADG" H -600 1900 50  0001 C CNN "Part number"
-	1    3300 4800
+	2    3300 4800
 	-1   0    0    1
 $EndComp

Commit message: Finish silkscreen
Parts:
- C224: value 220p -> 2.2n; Part number ECHU1H221GX5 -> ECHU1H222GX5
- U201, U204: Part number NE5534ADG -> NE5532DR
- U202: Part number (none) -> NE5534ADG
Changed lines of the file:
@@
 AR Path="/5C7379E1/5C88EE9E" Ref="C324"  Part="1"
 F 0 "C224" H 7050 3600 50  0000 L CNN
-F 1 "220p" H 7050 3500 50  0000 L CNN
+F 1 "2.2n" H 7050 3500 50  0000 L CNN
 F 2 "actidamp-mk4-smd:C_0805_2012Metric_Pad1.15x1.1mm_HandSolder" H 7388 3400 50  0001 C CNN
 F 3 "~" H 7350 3550 50  0001 C CNN
-F 4 "ECHU1H221GX5" H 0   0   50  0001 C CNN "Part number"
+F 4 "ECHU1H222GX5" H 0   0   50  0001 C CNN "Part number"
 F 5 "PPS 0805" H 0   0   50  0001 C CNN "Parameters"
 	1    7350 3550
@@
 F 2 "Package_SO:SOIC-8_3.9x4.9mm_P1.27mm" H 3900 2900 50  0001 C CNN
 F 3 "http://www.farnell.com/datasheets/2160703.pdf" H 3900 2900 50  0001 C CNN
-F 4 "NE5534ADG" H 0   0   50  0001 C CNN "Part number"
+F 4 "NE5532DR" H 0   0   50  0001 C CNN "Part number"
 	1    3900 2900
 	1    0    0    -1
@@
 F 2 "Package_SO:SOIC-8_3.9x4.9mm_P1.27mm" H 7850 3050 50  0001 C CNN
 F 3 "http://www.farnell.com/datasheets/2160703.pdf" H 7850 3050 50  0001 C CNN
-F 4 "NE5534ADG" H 0   0   50  0001 C CNN "Part number"
+F 4 "NE5532DR" H 0   0   50  0001 C CNN "Part number"
 	2    7850 3050
 	1    0    0    -1
@@
 F 2 "Package_SO:SOIC-8_3.9x4.9mm_P1.27mm" H 10100 2200 50  0001 C CNN
 F 3 "http://www.farnell.com/datasheets/2160703.pdf" H 10100 2200 50  0001 C CNN
-F 4 "NE5534ADG" H 0   -100 50  0001 C CNN "Part number"
+F 4 "NE5532DR" H 0   -100 50  0001 C CNN "Part number"
 	3    10100 2200
 	1    0    0    -1
@@
 F 2 "Package_SO:SOIC-8_3.9x4.9mm_P1.27mm" H 10000 3150 50  0001 C CNN
 F 3 "http://www.farnell.com/datasheets/2160703.pdf" H 10000 3150 50  0001 C CNN
-F 4 "NE5534ADG" H 0   0   50  0001 C CNN "Part number"
+F 4 "NE5532DR" H 0   0   50  0001 C CNN "Part number"
 	1    10000 3150
 	1    0    0    -1
@@
 F 2 "Package_SO:SOIC-8_3.9x4.9mm_P1.27mm" H 3300 4800 50  0001 C CNN
 F 3 "http://www.farnell.com/datasheets/2160703.pdf" H 3300 4800 50  0001 C CNN
-F 4 "NE5534ADG" H -600 1900 50  0001 C CNN "Part number"
+F 4 "NE5532DR" H -600 1900 50  0001 C CNN "Part number"
 	2    3300 4800
 	-1   0    0    1
@@
 F 2 "Package_SO:SOIC-8_3.9x4.9mm_P1.27mm" H 4000 1950 50  0001 C CNN
 F 3 "http://www.farnell.com/datasheets/2160703.pdf" H 4000 1950 50  0001 C CNN
-F 4 "NE5534ADG" H 0   -100 50  0001 C CNN "Part number"
+F 4 "NE5532DR" H 0   -100 50  0001 C CNN "Part number"
 	3    4000 1950
 	1    0    0    -1
@@
 F 2 "Package_SO:SOIC-8_3.9x4.9mm_P1.27mm" H 6200 2200 50  0001 C CNN
 F 3 "http://www.ti.com/lit/ds/symlink/ne5534.pdf" H 6200 2300 50  0001 C CNN
+F 4 "NE5534ADG" H 6150 2150 50  0001 C CNN "Part number"
 	1    6150 2150
 	1    0    0    -1
