File: actidamp-mk4-smd.kicad_pcb (KiCad board)
At the start: 2 copper layers, 159 x 120 mm, 203 parts, among them J101 XLR3, J102 Phono_Ground, J103 PHONO_IN_L, J104 PHONO_IN_R, J105 LINE_OUT_L, J106 LINE_OUT_R, Q201 2SK3320, Q301 2SK3320, Q401 BC846BPN, Q501 BC846BPN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

Commit message: All components placed on board
Parts:
- moved C226 288.6 mm to (107.0, -29.0), turned to 90 degrees
- moved C232 268.6 mm to (86.5, -26.0), turned to 270 degrees
- moved U205 266.2 mm to (99.5, -18.5), turned to 270 degrees
- moved C231 263.7 mm to (84.0, -26.0), turned to 270 degrees
- moved R224 262.4 mm to (92.6, -26.0), turned to 180 degrees
- moved R230 258.8 mm to (95.5, -21.6), turned to 90 degrees
- moved R229 258.4 mm to (93.0, -31.4), turned to 270 degrees
- moved C228 257.9 mm to (80.0, -29.5), turned to 180 degrees
- moved C229 254.3 mm to (98.5, -29.0), turned to 270 degrees
- moved C225 251.7 mm to (85.0, -29.5)
- moved C224 251.3 mm to (76.0, -26.0), turned to 90 degrees
- moved R403 247.0 mm to (113.5, -29.5), turned to 90 degrees
- moved R401 246.8 mm to (117.0, -29.5), turned to 90 degrees
- moved C103 246.6 mm to (100.5, 31.8)
- moved U204 246.6 mm to (90.5, -18.5), turned to 270 degrees
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Routing:
- net /right_channel/V-: track 0.00 -> 41.5 mm
- net /left_channel/V-: track 0.00 -> 41.5 mm
- net Net-(C218-Pad1): track 0.00 -> 37.3 mm
- net Net-(C218-Pad2): track 0.00 -> 34.4 mm
- net Net-(C226-Pad1): track 0.00 -> 28.2 mm
- net Net-(C502-Pad2): track 0.00 -> 27.9 mm, vias 0 -> 2
- net Net-(C402-Pad2): track 0.00 -> 27.9 mm, vias 0 -> 2
- net Net-(C225-Pad1): track 0.00 -> 24.2 mm
- net Net-(C216-Pad1): track 28.2 -> 4.95 mm
- net Net-(Q501-Pad6): track 0.00 -> 22.4 mm, vias 0 -> 2
- net Net-(Q401-Pad6): track 0.00 -> 22.4 mm, vias 0 -> 2
- net /psu_rails_left/Vreg+: track 0.00 -> 20.9 mm
- net Net-(C226-Pad2): track 0.00 -> 20.6 mm
- net Net-(C401-Pad1): track 0.00 -> 20.4 mm, vias 0 -> 2
- net Net-(C501-Pad1): track 0.00 -> 20.4 mm, vias 0 -> 2
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Other:
- board size 159 x 120 mm -> 119 x 100 mm

Commit message: More routing
Parts:
- removed H101, H102, H103, H104: MountingHole, MountingHole:MountingHole_2.7mm_M2.5
- moved R502 14.4 mm to (114.6, 18.2), turned to 270 degrees
- moved R402 13.9 mm to (115.0, -23.1), turned to 270 degrees
- moved C507 13.2 mm to (67.5, -2.19)
- moved R504 13.0 mm to (113.3, 4.31), turned to 180 degrees
- moved C407 12.5 mm to (67.9, -43.5)
- moved C106 12.5 mm to (82.5, 35.0), turned to 180 degrees
- moved R219 11.6 mm to (62.5, -43.5), turned to 0 degrees
- moved R404 11.0 mm to (113.6, -37.0)
- moved R319 10.6 mm to (63.7, -1.61), turned to 0 degrees
- moved R316 9.31 mm to (53.2, 15.0), turned to 270 degrees
- moved R213 9.14 mm to (58.0, -43.5)
- moved R220 9.00 mm to (51.5, -13.5), turned to 0 degrees
- moved R104 8.95 mm to (86.0, 41.1)
- moved R216 8.85 mm to (52.0, -26.9), turned to 270 degrees
- moved R501 8.81 mm to (112.1, 18.3), turned to 270 degrees
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Connections:
- J105 pad 3: (no net) -> Net-(J105-Pad3)
- J106 pad 3: (no net) -> Net-(J106-Pad3)
- U202 pad 1: (no net) -> Net-(U202-Pad1)
- U203 pad 1: (no net) -> Net-(U203-Pad1)
- U203 pad 5: (no net) -> Net-(U203-Pad5)
- U203 pad 8: (no net) -> Net-(U203-Pad8)
- U205 pad 8: (no net) -> Net-(U205-Pad8)
- U302 pad 1: (no net) -> Net-(U302-Pad1)
- U303 pad 1: (no net) -> Net-(U303-Pad1)
- U303 pad 5: (no net) -> Net-(U303-Pad5)
- U303 pad 8: (no net) -> Net-(U303-Pad8)
- U305 pad 8: (no net) -> Net-(U305-Pad8)
Routing:
- net /left_channel/V+: track 29.1 -> 152.9 mm, vias 2 -> 5
- net GND: track 40.6 -> 160.0 mm, vias 17 -> 66
- net /right_channel/V+: track 20.2 -> 88.2 mm, vias 0 -> 4
- net Net-(C313-Pad2): track 0.00 -> 60.7 mm
- net /left_channel/V-: track 41.5 -> 101.9 mm, vias 0 -> 5
- net /right_channel/V-: track 41.5 -> 86.4 mm, vias 0 -> 5
- net Net-(C318-Pad1): track 0.00 -> 39.6 mm
- net Net-(C316-Pad1): track 0.00 -> 36.9 mm
- net Net-(C318-Pad2): track 0.00 -> 36.7 mm
- net Net-(C312-Pad2): track 0.00 -> 33.0 mm
- net Net-(C216-Pad1): track 4.95 -> 36.9 mm
- net Net-(Q301-Pad3): track 0.00 -> 31.8 mm, vias 0 -> 2
- net Net-(R317-Pad1): track 0.00 -> 27.2 mm
- net Net-(C326-Pad1): track 0.00 -> 26.2 mm, vias 0 -> 2
- net Net-(C307-Pad1): track 0.00 -> 26.2 mm
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- added copper zone on B.Cu, net GND

Commit message: All routed
Parts:
- moved D103 152.5 mm to (199.5, 142.5)
- moved R103 151.1 mm to (199.0, 138.5), turned to 180 degrees
- moved C102 146.2 mm to (144.5, 142.5)
- moved D104 138.3 mm to (164.5, 133.0)
- moved C501 136.3 mm to (175.6, 109.3)
- moved C502 136.3 mm to (186.6, 98.3)
- moved C503 136.3 mm to (177.9, 102.3)
- moved C504 136.3 mm to (195.4, 102.3)
- moved C505 136.3 mm to (163.6, 98.8)
- moved C507 136.3 mm to (159.0, 98.8)
- moved C509 136.3 mm to (168.3, 98.8)
- moved Q501 136.3 mm to (187.1, 107.8)
- moved R501 136.3 mm to (203.6, 119.3)
- moved R502 136.3 mm to (206.1, 119.2)
- moved R503 136.3 mm to (203.6, 113.8)
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Routing:
- net /left_channel/V+: track 152.9 -> 25.1 mm, vias 5 -> 12
- net /right_channel/OUT: track 0.00 -> 104.1 mm, vias 0 -> 1
- net /left_channel/OUT: track 0.00 -> 86.9 mm, vias 0 -> 1
- net Net-(C101-Pad1): track 0.00 -> 83.2 mm
- net Net-(C102-Pad2): track 0.00 -> 67.9 mm
- net /right_channel/V+: track 88.2 -> 25.0 mm, vias 4 -> 12
- net /psu_rails_left/Vreg+: track 0.00 -> 45.6 mm, vias 0 -> 5
- net Net-(C501-Pad1): track 7.34 -> 40.8 mm, vias 2 -> 3
- net /left_channel/V-: track 101.9 -> 73.6 mm, vias 5 -> 11
- net Net-(C318-Pad1): track 39.6 -> 66.8 mm, vias 0 -> 2
- net /left_channel/IN: track 12.5 -> 32.3 mm
- net GND: track 160.0 -> 140.4 mm, vias 66 -> 75
- net /right_channel/IN: track 12.5 -> 28.1 mm
- net Net-(R317-Pad1): track 27.2 -> 42.5 mm, vias 0 -> 2
- net Net-(D103-Pad2): track 0.00 -> 14.1 mm
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- added copper zone on In2.Cu, net /left_channel/V+
- added copper zone on B.Cu, net /left_channel/V-
- added copper zone on In2.Cu, net /psu_rails_left/Vreg+
- added copper zone on B.Cu, net /psu_rails_left/Vreg-
- added copper zone on In2.Cu, net /right_channel/V+
- added copper zone on B.Cu, net /right_channel/V-
- added copper zone on In1.Cu, net GND
- removed copper zone on B.Cu, net GND
Other:
- copper layers 2 -> 4

Commit message: Finish silkscreen
Parts:
- moved R103 6.58 mm to (205.5, 139.5), turned to 0 degrees
- moved D103 6.00 mm to (205.5, 142.6), turned to 180 degrees
Routing:
- net Net-(D103-Pad2): track 14.1 -> 24.5 mm
- net /psu_rails_left/Vreg+: track 45.6 -> 51.1 mm, vias 5 -> 4
- net GND: track 140.4 -> 142.7 mm, vias 75 -> 74
Other:
- board text added: "Actidamp MK. IV by Pavel Dudek SMD version (C) Bruno Kremel"
- board text added: "IN L"
- board text added: "IN R"
- board text added: "OUT L"
- board text added: "OUT R"
- board text added: "POWER"
