File: psu-brick/psu-brick.sch (KiCad schematic (older format))
At the start: 16 parts, among them J1 Conn_01x02, J2 Conn_01x03

Commit message: Finish PSU brick
Parts:
- removed TR1: TRANSF3, symbol Transformer:TRANSF3
- added H1, H2, H3, H4: MountingHole, MountingHole:MountingHole_3.5mm, symbol Mechanical:MountingHole
- added TR1: TRANSF3_MYRRA, actidamp-mk4-smd:Transformer_Myrra_44x, symbol actidamp:TRANSF3_MYRRA
- C1: footprint (none) -> Capacitor_THT:C_Rect_L7.2mm_W7.2mm_P5.00mm_FKS2_FKP2_MKS2_MKP2; Part number (none) -> MKP2J016801C00KSSD
- C2, C3, C4, C5: footprint (none) -> Capacitor_SMD:C_0805_2012Metric_Pad1.15x1.40mm_HandSolder; Parameters (none) -> 0805
- C6, C7: footprint (none) -> Capacitor_THT:CP_Radial_D16.0mm_P7.50mm; symbol Device:C -> Device:CP; Parameters (none) -> Radial electrolytic (7.5mm)
- D1: footprint (none) -> actidamp-mk4-smd:MDB6S; Parameters (none) -> 1A
- D2: footprint (none) -> LED_THT:LED_D5.0mm; Part number (none) -> LTL2R3KRD-EM
- F1, F2: footprint (none) -> Fuse:Fuseholder_Cylinder-5x20mm_Schurter_0031_8201_Horizontal_Open; Part number (none) -> 0031.8201
- J1: value Conn_01x02 -> 230V AC; footprint (none) -> actidamp-mk4-smd:AC_entry_770W-X2; Part number (none) -> 770W-X2/10
- J2: value Conn_01x03 -> +/- 34V DC; footprint (none) -> TerminalBlock_TE-Connectivity:TerminalBlock_TE_282834-3_1x03_P2.54mm_Horizontal
- R1, R2: footprint (none) -> Resistor_SMD:R_1206_3216Metric_Pad1.42x1.75mm_HandSolder; Parameters (none) -> 1206
Connections:
- net GND: now also TR1.7, TR1.9
- net at C1.1, J1.2 (Pin_2): now also TR1.1
- net at C1.2, J1.1 (Pin_1): now also TR1.5
- net at F1.2: now also TR1.6
- net at F2.2: now also TR1.10
Other:
- moved on the sheet: C2, C3, C4, C5, R1, R2
