File: psu-brick/psu-brick.kicad_pcb (KiCad board)
At the start: 2 copper layers, 114 x 60 mm, 20 parts, among them J1 230V AC, J2 +/- 34V DC

Commit message: Fix unconnected wire
Routing:
- net Net-(C2-Pad2): track 30.9 -> 36.4 mm
Changed lines of the file:
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@@
     (thickness 1.6)
     (drawings 16)
-    (tracks 100)
+    (tracks 103)
     (zones 0)
     (modules 20)
@@
     (visible_elements 7FFFFFFF)
     (pcbplotparams
-      (layerselection 0x010fc_ffffffff)
+      (layerselection 0x010f0_ffffffff)
       (usegerberextensions false)
       (usegerberattributes false)
@@
       (outputformat 1)
       (mirror false)
-      (drillshape 1)
+      (drillshape 0)
       (scaleselection 1)
-      (outputdirectory ""))
+      (outputdirectory "./gerbers"))
   )
   (net 0 "")
@@
   (segment (start 120.975001 99.400001) (end 120 98.425) (width 0.7) (layer F.Cu) (net 4))
   (segment (start 120.975001 102.015003) (end 120.975001 99.400001) (width 0.7) (layer F.Cu) (net 4))
-  (segment (start 129.459999 110.500001) (end 120.975001 102.015003) (width 0.7) (layer F.Cu) (net 4))
   (segment (start 131.500001 110.500001) (end 129.459999 110.500001) (width 0.7) (layer F.Cu) (net 4))
   (segment (start 133 112) (end 131.500001 110.500001) (width 0.7) (layer F.Cu) (net 4))
+  (segment (start 127.129999 103.920001) (end 128 103.05) (width 0.7) (layer F.Cu) (net 4))
+  (segment (start 127.129999 108.170001) (end 127.129999 103.920001) (width 0.7) (layer F.Cu) (net 4))
+  (segment (start 129.459999 110.500001) (end 127.129999 108.170001) (width 0.7) (layer F.Cu) (net 4))
+  (segment (start 127.129999 108.170001) (end 120.975001 102.015003) (width 0.7) (layer F.Cu) (net 4))
   (segment (start 125.85 101) (end 124 102.85) (width 0.7) (layer F.Cu) (net 5))
   (segment (start 128 101) (end 125.85 101) (width 0.7) (layer F.Cu) (net 5))
