File: main-pcb/actidamp-mk4-smd.sch (KiCad schematic (older format))
At the start: 24 parts, among them J101 XLR3, J102 Phono_Ground, J103 PHONO_IN_L, J104 PHONO_IN_R, J105 LINE_OUT_L, J106 LINE_OUT_R, U101 LM317_3PinPackage, U102 LM337_TO252

Commit message: Some minor modifications
Other:
- note added: "Input in range of +-25 up to +-28V"
- note removed: "Input in range of +-25 up to +-35V"
Changed lines of the file:
@@
 The output of regulators should be +- approx. 18.5\nThat makes +- approx. 17.5 after psu_rails capacitor multiplier
 Text Notes 1300 4000 1    50   ~ 0
-Input in range of +-25 up to +-35V
+Input in range of +-25 up to +-28V
 Wire Wire Line
 	8100 2650 8100 3800
